File: portable-line-mixer.sch (KiCad schematic (older format))
At the start: 17 parts

Commit message: finished with first draft of schematic
Parts:
- gave numbers to parts that had none: 15
Connections:
- net GNDREF: now also U1.3 (+), U1.5 (+); no longer U1.3 (+), U1.5 (+)
- net Stereo-Input-0/LOUT: now also U1.6 (-); no longer U1.2 (-)
- net Stereo-Input-0/ROUT: now also U1.2 (-); no longer U1.6 (-)
- net at C2.2, C3.1, R2.1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: now also U1.7 (OUT); no longer U1.1 (OUT)
- net at C1.2, C4.1, R1.1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: now also U1.1 (OUT); no longer U1.7 (OUT)
- no-connect marks 0 -> 1
Other:
- note added: "Potential connection\nfor an LCD display"
Changed lines of the file:
@@
 EESchema Schematic File Version 2
+LIBS:SW-Linear
 LIBS:SW-IQD
 LIBS:SW-NXP
@@
 Connection ~ 4600 3400
 $Comp
-L RC4560 U?
-U 1 1 580B2CB5
+L RC4560 U1
+U 2 1 580B2CB5
 P 3550 5450
-F 0 "U?" H 3500 5350 60  0000 C CNN
+F 0 "U1" H 3500 5350 60  0000 C CNN
 F 1 "RC4560" H 3600 5450 60  0000 C CNN
 F 2 "" H 3600 5450 60  0000 C CNN
@@
 F 9 "Texas Instruments" H 3800 5650 60  0001 C CNN "Manufacturer"
 F 10 "The RC4560 is a high-gain, wide-bandwidth, dual operational amplifier capable of driving 20 V peak-to-peak into 400-Ω loads" H 3700 5550 60  0001 C CNN "Description"
-	1    3550 5450
+	2    3550 5450
 	1    0    0    1
 $EndComp
 $Comp
-L RC4560 U?
-U 2 1 580B3637
+L RC4560 U1
+U 1 1 580B3637
 P 3500 6950
-F 0 "U?" H 3450 6850 60  0000 C CNN
+F 0 "U1" H 3450 6850 60  0000 C CNN
 F 1 "RC4560" H 3550 6950 60  0000 C CNN
 F 2 "" H 3550 6950 60  0000 C CNN
@@
 F 9 "Texas Instruments" H 3750 7150 60  0001 C CNN "Manufacturer"
 F 10 "The RC4560 is a high-gain, wide-bandwidth, dual operational amplifier capable of driving 20 V peak-to-peak into 400-Ω loads" H 3650 7050 60  0001 C CNN "Description"
-	2    3500 6950
+	1    3500 6950
 	1    0    0    1
 $EndComp
 $Comp
-L RC4560 U?
+L RC4560 U2
 U 1 1 580B3FF5
 P 5100 5600
-F 0 "U?" H 5050 5500 60  0000 C CNN
+F 0 "U2" H 5050 5500 60  0000 C CNN
 F 1 "RC4560" H 5150 5600 60  0000 C CNN
 F 2 "" H 5150 5600 60  0000 C CNN
@@
 $EndComp
 $Comp
-L RC4560 U?
+L RC4560 U2
 U 2 1 580B5187
 P 5100 7100
-F 0 "U?" H 5050 7000 60  0000 C CNN
+F 0 "U2" H 5050 7000 60  0000 C CNN
 F 1 "RC4560" H 5150 7100 60  0000 C CNN
 F 2 "" H 5150 7100 60  0000 C CNN
@@
 Connection ~ 3000 4350
 $Comp
-L R R?
+L R R2
 U 1 1 580B7023
 P 3600 4800
-F 0 "R?" V 3680 4800 50  0000 C CNN
+F 0 "R2" V 3680 4800 50  0000 C CNN
 F 1 "10k" V 3600 4800 50  0000 C CNN
 F 2 "" V 3530 4800 50  0000 C CNN
@@
 $EndComp
 $Comp
-L R R?
+L R R3
 U 1 1 580B71E8
 P 5150 4950
-F 0 "R?" V 5230 4950 50  0000 C CNN
+F 0 "R3" V 5230 4950 50  0000 C CNN
 F 1 "10k" V 5150 4950 50  0000 C CNN
 F 2 "" V 5080 4950 50  0000 C CNN
@@
 $EndComp
 $Comp
-L C C?
+L C C2
 U 1 1 580B7BF4
 P 3600 4600
-F 0 "C?" H 3625 4700 50  0000 L CNN
+F 0 "C2" H 3625 4700 50  0000 L CNN
 F 1 "27pF" H 3625 4500 50  0000 L CNN
 F 2 "" H 3638 4450 50  0000 C CNN
@@
 $EndComp
 $Comp
-L C C?
+L C C3
 U 1 1 580B8B1D
 P 5150 4800
-F 0 "C?" H 5175 4900 50  0000 L CNN
+F 0 "C3" H 5175 4900 50  0000 L CNN
 F 1 "47pF" H 5175 4700 50  0000 L CNN
 F 2 "" H 5188 4650 50  0000 C CNN
@@
 	4150 4800 4150 5450
 $Comp
-L R R?
+L R R1
 U 1 1 580BA60C
 P 3550 6350
-F 0 "R?" V 3630 6350 50  0000 C CNN
+F 0 "R1" V 3630 6350 50  0000 C CNN
 F 1 "10k" V 3550 6350 50  0000 C CNN
 F 2 "" V 3480 6350 50  0000 C CNN
@@
 $EndComp
 $Comp
-L C C?
+L C C1
 U 1 1 580BA612
 P 3550 6200
-F 0 "C?" H 3575 6300 50  0000 L CNN
+F 0 "C1" H 3575 6300 50  0000 L CNN
 F 1 "27pF" H 3575 6100 50  0000 L CNN
 F 2 "" H 3588 6050 50  0000 C CNN
@@
 	5700 4950 5700 5600
 $Comp
-L R R?
+L R R4
 U 1 1 580BC069
 P 5150 6450
-F 0 "R?" V 5230 6450 50  0000 C CNN
+F 0 "R4" V 5230 6450 50  0000 C CNN
 F 1 "10k" V 5150 6450 50  0000 C CNN
 F 2 "" V 5080 6450 50  0000 C CNN
@@
 $EndComp
 $Comp
-L C C?
+L C C4
 U 1 1 580BC06F
 P 5150 6250
-F 0 "C?" H 5175 6350 50  0000 L CNN
+F 0 "C4" H 5175 6350 50  0000 L CNN
 F 1 "47pF" H 5175 6150 50  0000 L CNN
 F 2 "" H 5188 6100 50  0000 C CNN
@@
 	4700 6950 4100 6950
 $Comp
-L -12VA #PWR?
+L -12VA #PWR015
 U 1 1 580BCC5B
 P 3600 5100
-F 0 "#PWR?" H 3600 4950 50  0001 C CNN
+F 0 "#PWR015" H 3600 4950 50  0001 C CNN
 F 1 "-12VA" H 3600 5240 50  0000 C CNN
 F 2 "" H 3600 5100 50  0000 C CNN
@@
 $EndComp
 $Comp
-L -12VA #PWR?
+L -12VA #PWR016
 U 1 1 580BD87D
 P 3550 6600
-F 0 "#PWR?" H 3550 6450 50  0001 C CNN
+F 0 "#PWR016" H 3550 6450 50  0001 C CNN
 F 1 "-12VA" H 3550 6740 50  0000 C CNN
 F 2 "" H 3550 6600 50  0000 C CNN
@@
 $EndComp
 $Comp
-L -12VA #PWR?
+L -12VA #PWR017
 U 1 1 580BDA2F
 P 5150 6750
-F 0 "#PWR?" H 5150 6600 50  0001 C CNN
+F 0 "#PWR017" H 5150 6600 50  0001 C CNN
 F 1 "-12VA" H 5150 6890 50  0000 C CNN
 F 2 "" H 5150 6750 50  0000 C CNN
@@
 $EndComp
 $Comp
-L -12VA #PWR?
+L -12VA #PWR018
 U 1 1 580BEB7A
 P 5150 5250
-F 0 "#PWR?" H 5150 5100 50  0001 C CNN
+F 0 "#PWR018" H 5150 5100 50  0001 C CNN
 F 1 "-12VA" H 5150 5390 50  0000 C CNN
 F 2 "" H 5150 5250 50  0000 C CNN
@@
 $EndComp
 $Comp
-L +12VA #PWR?
+L +12VA #PWR019
 U 1 1 580BF2C0
 P 3550 7300
-F 0 "#PWR?" H 3550 7150 50  0001 C CNN
+F 0 "#PWR019" H 3550 7150 50  0001 C CNN
 F 1 "+12VA" H 3550 7440 50  0000 C CNN
 F 2 "" H 3550 7300 50  0000 C CNN
@@
 $EndComp
 $Comp
-L +12VA #PWR?
+L +12VA #PWR020
 U 1 1 580BF479
 P 5150 7450
-F 0 "#PWR?" H 5150 7300 50  0001 C CNN
+F 0 "#PWR020" H 5150 7300 50  0001 C CNN
 F 1 "+12VA" H 5150 7590 50  0000 C CNN
 F 2 "" H 5150 7450 50  0000 C CNN
@@
 $EndComp
 $Comp
-L +12VA #PWR?
+L +12VA #PWR021
 U 1 1 580BF62B
 P 5150 5950
-F 0 "#PWR?" H 5150 5800 50  0001 C CNN
+F 0 "#PWR021" H 5150 5800 50  0001 C CNN
 F 1 "+12VA" H 5150 6090 50  0000 C CNN
 F 2 "" H 5150 5950 50  0000 C CNN
@@
 $EndComp
 $Comp
-L +12VA #PWR?
+L +12VA #PWR022
 U 1 1 580BF7DD
 P 3600 5800
-F 0 "#PWR?" H 3600 5650 50  0001 C CNN
+F 0 "#PWR022" H 3600 5650 50  0001 C CNN
 F 1 "+12VA" H 3600 5940 50  0000 C CNN
 F 2 "" H 3600 5800 50  0000 C CNN
@@
 $EndComp
 $Comp
-L GNDREF #PWR?
+L GNDREF #PWR023
 U 1 1 580C026A
 P 3150 5600
-F 0 "#PWR?" H 3150 5350 50  0001 C CNN
+F 0 "#PWR023" H 3150 5350 50  0001 C CNN
 F 1 "GNDREF" H 3150 5450 50  0000 C CNN
 F 2 "" H 3150 5600 50  0000 C CNN
@@
 $EndComp
 $Comp
-L GNDREF #PWR?
+L GNDREF #PWR024
 U 1 1 580C067D
 P 3100 7100
-F 0 "#PWR?" H 3100 6850 50  0001 C CNN
+F 0 "#PWR024" H 3100 6850 50  0001 C CNN
 F 1 "GNDREF" H 3100 6950 50  0000 C CNN
 F 2 "" H 3100 7100 50  0000 C CNN
@@
 $EndComp
 $Comp
-L GNDREF #PWR?
+L GNDREF #PWR025
 U 1 1 580C082C
 P 4700 7250
-F 0 "#PWR?" H 4700 7000 50  0001 C CNN
+F 0 "#PWR025" H 4700 7000 50  0001 C CNN
 F 1 "GNDREF" H 4700 7100 50  0000 C CNN
 F 2 "" H 4700 7250 50  0000 C CNN
@@
 $EndComp
 $Comp
-L GNDREF #PWR?
+L GNDREF #PWR026
 U 1 1 580C09DB
 P 4700 5750
-F 0 "#PWR?" H 4700 5500 50  0001 C CNN
+F 0 "#PWR026" H 4700 5500 50  0001 C CNN
 F 1 "GNDREF" H 4700 5600 50  0000 C CNN
 F 2 "" H 4700 5750 50  0000 C CNN
@@
 Connection ~ 2900 4250
 $Comp
-L JACK-TRS J?
+L JACK-TRS J1
 U 1 1 580C183E
 P 6850 5900
-F 0 "J?" H 6850 5800 60  0000 C CNN
+F 0 "J1" H 6850 5800 60  0000 C CNN
 F 1 "JACK-TRS" H 6850 5900 60  0000 C CNN
 F 2 "" H 6850 5900 60  0000 C CNN
@@
 $EndComp
 $Comp
-L R R?
+L R R5
 U 1 1 580C1AD0
 P 5950 5950
-F 0 "R?" V 6030 5950 50  0000 C CNN
+F 0 "R5" V 6030 5950 50  0000 C CNN
 F 1 "100R" V 5950 5950 50  0000 C CNN
 F 2 "" V 5880 5950 50  0000 C CNN
@@
 	6600 5950 6450 5950
 $Comp
-L C C?
+L C C5
 U 1 1 580C1EDB
 P 6300 5950
-F 0 "C?" H 6325 6050 50  0000 L CNN
+F 0 "C5" H 6325 6050 50  0000 L CNN
 F 1 "10uF" H 6325 5850 50  0000 L CNN
 F 2 "" H 6338 5800 50  0000 C CNN
@@
 	5800 5600 5700 5600
 $Comp
-L C C?
+L C C6
 U 1 1 580C49A9
 P 6300 6150
-F 0 "C?" H 6325 6250 50  0000 L CNN
+F 0 "C6" H 6325 6250 50  0000 L CNN
 F 1 "10uF" H 6325 6050 50  0000 L CNN
 F 2 "" H 6338 6000 50  0000 C CNN
@@
 $EndComp
 $Comp
-L R R?
+L R R6
 U 1 1 580C4B6A
 P 5950 6150
-F 0 "R?" V 6030 6150 50  0000 C CNN
+F 0 "R6" V 6030 6150 50  0000 C CNN
 F 1 "100R" V 5950 6150 50  0000 C CNN
 F 2 "" V 5880 6150 50  0000 C CNN
@@
 Connection ~ 5700 6450
 $Comp
-L GNDREF #PWR?
+L GNDREF #PWR027
 U 1 1 580C5655
 P 6600 6300
-F 0 "#PWR?" H 6600 6050 50  0001 C CNN
+F 0 "#PWR027" H 6600 6050 50  0001 C CNN
 F 1 "GNDREF" H 6600 6150 50  0000 C CNN
 F 2 "" H 6600 6300 50  0000 C CNN
@@
 F0 "Microprocessor" 60
 F1 "microprocessor.sch" 60
+F2 "SDA" B L 8150 4300 60
+F3 "SCL" B L 8150 4450 60
+F4 "~CE" B L 8150 4600 60
+F5 "TXserial" B R 9450 4400 60
 $EndSheet
+Text Label 3400 850  0    60   ~ 0
+SDA
+Text Label 3400 950  0    60   ~ 0
+SCL
+Text Label 3400 1050 0    60   ~ 0
+~CE
+Text Label 7900 4300 2    60   ~ 0
+SDA
+Text Label 7900 4450 2    60   ~ 0
+SCL
+Text Label 7900 4600 2    60   ~ 0
+~CE
+Wire Wire Line
+	8150 4300 7900 4300
+Wire Wire Line
+	7900 4450 8150 4450
+Wire Wire Line
+	8150 4600 7900 4600
+NoConn ~ 9450 4400
+Text Notes 9500 4350 0    60   ~ 0
+Potential connection\nfor an LCD display
 $EndSCHEMATC

Commit message: finalized schematic, finishing footprint assignment, starting pcb layout
Parts:
- removed C5, C6: 10uF, symbol C
- added C5, C6: 10uF, Capacitors_Tantalum_SMD:TantalC_SizeR_EIA-2012, symbol CP_Small
- C1, C2, C3, C4: footprint (none) -> Capacitors_SMD:C_0805_HandSoldering
- J1: footprint (none) -> SW-KYCON:STX-3100-3C
- R1, R2, R3, R4, R5, R6: footprint (none) -> Resistors_SMD:R_0805_HandSoldering
- U1, U2: footprint (none) -> Housings_SSOP:TSSOP-8_4.4x3mm_Pitch0.65mm
Connections:
- net at J1.2: now also C5.2
- net at J1.3: now also C6.2
- net at R5.1: now also C5.1
- net at R6.1: now also C6.1
Changed lines of the file:
@@
 F 0 "U1" H 3500 5350 60  0000 C CNN
 F 1 "RC4560" H 3600 5450 60  0000 C CNN
-F 2 "" H 3600 5450 60  0000 C CNN
+F 2 "Housings_SSOP:TSSOP-8_4.4x3mm_Pitch0.65mm" H 3600 5450 60  0001 C CNN
 F 3 "http://www.ti.com/lit/ds/symlink/rc4560.pdf" H 3600 5450 60  0001 C CNN
 F 4 "Any" H 3550 5450 60  0001 C CNN "Source"
@@
 F 0 "U1" H 3450 6850 60  0000 C CNN
 F 1 "RC4560" H 3550 6950 60  0000 C CNN
-F 2 "" H 3550 6950 60  0000 C CNN
+F 2 "Housings_SSOP:TSSOP-8_4.4x3mm_Pitch0.65mm" H 3550 6950 60  0001 C CNN
 F 3 "http://www.ti.com/lit/ds/symlink/rc4560.pdf" H 3550 6950 60  0001 C CNN
 F 4 "Any" H 3500 6950 60  0001 C CNN "Source"
@@
 F 0 "U2" H 5050 5500 60  0000 C CNN
 F 1 "RC4560" H 5150 5600 60  0000 C CNN
-F 2 "" H 5150 5600 60  0000 C CNN
+F 2 "Housings_SSOP:TSSOP-8_4.4x3mm_Pitch0.65mm" H 5150 5600 60  0001 C CNN
 F 3 "http://www.ti.com/lit/ds/symlink/rc4560.pdf" H 5150 5600 60  0001 C CNN
 F 4 "Any" H 5100 5600 60  0001 C CNN "Source"
@@
 F 0 "U2" H 5050 7000 60  0000 C CNN
 F 1 "RC4560" H 5150 7100 60  0000 C CNN
-F 2 "" H 5150 7100 60  0000 C CNN
+F 2 "Housings_SSOP:TSSOP-8_4.4x3mm_Pitch0.65mm" H 5150 7100 60  0001 C CNN
 F 3 "http://www.ti.com/lit/ds/symlink/rc4560.pdf" H 5150 7100 60  0001 C CNN
 F 4 "Any" H 5100 7100 60  0001 C CNN "Source"
@@
 F 0 "R2" V 3680 4800 50  0000 C CNN
 F 1 "10k" V 3600 4800 50  0000 C CNN
-F 2 "" V 3530 4800 50  0000 C CNN
+F 2 "Resistors_SMD:R_0805_HandSoldering" V 3530 4800 50  0001 C CNN
 F 3 "" H 3600 4800 50  0000 C CNN
 	1    3600 4800
@@
 F 0 "R3" V 5230 4950 50  0000 C CNN
 F 1 "10k" V 5150 4950 50  0000 C CNN
-F 2 "" V 5080 4950 50  0000 C CNN
+F 2 "Resistors_SMD:R_0805_HandSoldering" V 5080 4950 50  0001 C CNN
 F 3 "" H 5150 4950 50  0000 C CNN
 	1    5150 4950
@@
 F 0 "C2" H 3625 4700 50  0000 L CNN
 F 1 "27pF" H 3625 4500 50  0000 L CNN
-F 2 "" H 3638 4450 50  0000 C CNN
+F 2 "Capacitors_SMD:C_0805_HandSoldering" H 3638 4450 50  0001 C CNN
 F 3 "" H 3600 4600 50  0000 C CNN
 	1    3600 4600
@@
 F 0 "C3" H 5175 4900 50  0000 L CNN
 F 1 "47pF" H 5175 4700 50  0000 L CNN
-F 2 "" H 5188 4650 50  0000 C CNN
+F 2 "Capacitors_SMD:C_0805_HandSoldering" H 5188 4650 50  0001 C CNN
 F 3 "" H 5150 4800 50  0000 C CNN
 	1    5150 4800
@@
 F 0 "R1" V 3630 6350 50  0000 C CNN
 F 1 "10k" V 3550 6350 50  0000 C CNN
-F 2 "" V 3480 6350 50  0000 C CNN
+F 2 "Resistors_SMD:R_0805_HandSoldering" V 3480 6350 50  0001 C CNN
 F 3 "" H 3550 6350 50  0000 C CNN
 	1    3550 6350
@@
 F 0 "C1" H 3575 6300 50  0000 L CNN
 F 1 "27pF" H 3575 6100 50  0000 L CNN
-F 2 "" H 3588 6050 50  0000 C CNN
+F 2 "Capacitors_SMD:C_0805_HandSoldering" H 3588 6050 50  0001 C CNN
 F 3 "" H 3550 6200 50  0000 C CNN
 	1    3550 6200
@@
 F 0 "R4" V 5230 6450 50  0000 C CNN
 F 1 "10k" V 5150 6450 50  0000 C CNN
-F 2 "" V 5080 6450 50  0000 C CNN
+F 2 "Resistors_SMD:R_0805_HandSoldering" V 5080 6450 50  0001 C CNN
 F 3 "" H 5150 6450 50  0000 C CNN
 	1    5150 6450
@@
 F 0 "C4" H 5175 6350 50  0000 L CNN
 F 1 "47pF" H 5175 6150 50  0000 L CNN
-F 2 "" H 5188 6100 50  0000 C CNN
+F 2 "Capacitors_SMD:C_0805_HandSoldering" H 5188 6100 50  0001 C CNN
 F 3 "" H 5150 6250 50  0000 C CNN
 	1    5150 6250
@@
 F 0 "J1" H 6850 5800 60  0000 C CNN
 F 1 "JACK-TRS" H 6850 5900 60  0000 C CNN
-F 2 "" H 6850 5900 60  0000 C CNN
+F 2 "SW-KYCON:STX-3100-3C" H 6850 5900 60  0001 C CNN
 F 3 "" H 6850 5900 60  0000 C CNN
 	1    6850 5900
@@
 F 0 "R5" V 6030 5950 50  0000 C CNN
 F 1 "100R" V 5950 5950 50  0000 C CNN
-F 2 "" V 5880 5950 50  0000 C CNN
+F 2 "Resistors_SMD:R_0805_HandSoldering" V 5880 5950 50  0001 C CNN
 F 3 "" H 5950 5950 50  0000 C CNN
 	1    5950 5950
@@
 $EndComp
 Wire Wire Line
-	6600 5950 6450 5950
-$Comp
-L C C5
-U 1 1 580C1EDB
-P 6300 5950
-F 0 "C5" H 6325 6050 50  0000 L CNN
-F 1 "10uF" H 6325 5850 50  0000 L CNN
-F 2 "" H 6338 5800 50  0000 C CNN
-F 3 "" H 6300 5950 50  0000 C CNN
-	1    6300 5950
-	0    1    1    0
-$EndComp
-Wire Wire Line
-	6150 5950 6100 5950
+	6400 5950 6600 5950
+Wire Wire Line
+	6100 5950 6200 5950
 Wire Wire Line
 	5800 5950 5800 5600
 Wire Wire Line
 	5800 5600 5700 5600
-$Comp
-L C C6
-U 1 1 580C49A9
-P 6300 6150
-F 0 "C6" H 6325 6250 50  0000 L CNN
-F 1 "10uF" H 6325 6050 50  0000 L CNN
-F 2 "" H 6338 6000 50  0000 C CNN
-F 3 "" H 6300 6150 50  0000 C CNN
-	1    6300 6150
-	0    1    1    0
-$EndComp
 $Comp
 L R R6
@@
 F 0 "R6" V 6030 6150 50  0000 C CNN
 F 1 "100R" V 5950 6150 50  0000 C CNN
-F 2 "" V 5880 6150 50  0000 C CNN
+F 2 "Resistors_SMD:R_0805_HandSoldering" V 5880 6150 50  0001 C CNN
 F 3 "" H 5950 6150 50  0000 C CNN
 	1    5950 6150
@@
 $EndComp
 Wire Wire Line
-	6150 6150 6100 6150
-Wire Wire Line
-	6450 6150 6600 6150
+	6100 6150 6200 6150
+Wire Wire Line
+	6400 6150 6600 6150
 Wire Wire Line
 	5800 6450 5800 6150
@@
 Text Notes 9500 4350 0    60   ~ 0
 Potential connection\nfor an LCD display
+$Comp
+L CP_Small C5
+U 1 1 5813E56A
+P 6300 5950
+F 0 "C5" H 6310 6020 50  0000 L CNN
+F 1 "10uF" H 6310 5870 50  0000 L CNN
+F 2 "Capacitors_Tantalum_SMD:TantalC_SizeR_EIA-2012" H 6300 5950 50  0001 C CNN
+F 3 "" H 6300 5950 50  0000 C CNN
+	1    6300 5950
+	0    -1   -1   0
+$EndComp
+$Comp
+L CP_Small C6
+U 1 1 5813FB41
+P 6300 6150
+F 0 "C6" H 6310 6220 50  0000 L CNN
+F 1 "10uF" H 6310 6070 50  0000 L CNN
+F 2 "Capacitors_Tantalum_SMD:TantalC_SizeR_EIA-2012" H 6300 6150 50  0001 C CNN
+F 3 "" H 6300 6150 50  0000 C CNN
+	1    6300 6150
+	0    -1   -1   0
+$EndComp
 $EndSCHEMATC

Commit message: replacing audio jack footprints
Parts:
- J1: footprint SW-KYCON:STX-3100-3C -> SW-CUI-INC:SJ1-353XNG-3Pin
Changed lines of the file:
@@
 F 0 "J1" H 6850 5800 60  0000 C CNN
 F 1 "JACK-TRS" H 6850 5900 60  0000 C CNN
-F 2 "SW-KYCON:STX-3100-3C" H 6850 5900 60  0001 C CNN
+F 2 "SW-CUI-INC:SJ1-353XNG-3Pin" H 6850 5900 60  0001 C CNN
 F 3 "" H 6850 5900 60  0000 C CNN
 	1    6850 5900

Commit message: before initial DRC
Parts:
- added R34, R35: 4k7, Capacitors_SMD:C_0805_HandSoldering, symbol R
Connections:
- net +5VD: now also R34.2, R35.2
- net SCL: now also R35.1
- net SDA: now also R34.1
Changed lines of the file:
@@
 ~CE
 Wire Wire Line
-	8150 4300 7900 4300
+	7700 4300 8150 4300
 Wire Wire Line
-	7900 4450 8150 4450
+	7700 4450 8150 4450
 Wire Wire Line
 	8150 4600 7900 4600
@@
 	0    -1   -1   0
 $EndComp
+$Comp
+L R R34
+U 1 1 5815B213
+P 7550 4300
+F 0 "R34" V 7630 4300 50  0000 C CNN
+F 1 "4k7" V 7550 4300 50  0000 C CNN
+F 2 "Capacitors_SMD:C_0805_HandSoldering" V 7480 4300 50  0001 C CNN
+F 3 "" H 7550 4300 50  0000 C CNN
+	1    7550 4300
+	0    1    1    0
+$EndComp
+$Comp
+L R R35
+U 1 1 5815B4D4
+P 7550 4450
+F 0 "R35" V 7630 4450 50  0000 C CNN
+F 1 "4k7" V 7550 4450 50  0000 C CNN
+F 2 "Capacitors_SMD:C_0805_HandSoldering" V 7480 4450 50  0001 C CNN
+F 3 "" H 7550 4450 50  0000 C CNN
+	1    7550 4450
+	0    1    1    0
+$EndComp
+Wire Wire Line
+	7400 4300 7350 4300
+Wire Wire Line
+	7350 4300 7350 4450
+Wire Wire Line
+	7350 4450 7400 4450
+$Comp
+L +5VD #PWR028
+U 1 1 5815BF9A
+P 7350 4300
+F 0 "#PWR028" H 7350 4150 50  0001 C CNN
+F 1 "+5VD" H 7350 4440 50  0000 C CNN
+F 2 "" H 7350 4300 50  0000 C CNN
+F 3 "" H 7350 4300 50  0000 C CNN
+	1    7350 4300
+	1    0    0    -1
+$EndComp
 $EndSCHEMATC
