File: stereo-input.sch (KiCad schematic (older format))
At the start: 9 parts

Commit message: finished with first draft of schematic
Parts:
- gave numbers to parts that had none: 9
Connections:
- net +5VD: now also C10.2
- net -5V: now also C7.1
- net GNDREF: now also C7.2

Commit message: finalized schematic, finishing footprint assignment, starting pcb layout
Parts:
- C10, C11, C7, C8, C9: footprint (none) -> Capacitors_SMD:C_0603_HandSoldering
- J2: footprint (none) -> SW-KYCON:STX-3100-3C
- R7, R8: footprint (none) -> Resistors_SMD:R_0805_HandSoldering
- U3: footprint (none) -> Housings_SSOP:TSSOP-16_4.4x5mm_Pitch0.65mm
Changed lines of the file:
@@
 AR Path="/580A1257/5809B3AA" Ref="U9"  Part="1"
 AR Path="/580A1261/5809B3AA" Ref="U10"  Part="1"
-F 0 "U3" V 3300 2400 60  0000 C CNN
+F 0 "U7" V 3300 2400 60  0000 C CNN
 F 1 "DS1882" V 3300 2000 60  0000 C CNN
-F 2 "" H 3200 2300 60  0001 C CNN
+F 2 "Housings_SSOP:TSSOP-16_4.4x5mm_Pitch0.65mm" H 3200 2300 60  0001 C CNN
 F 3 "https://datasheets.maximintegrated.com/en/ds/DS1882.pdf" H 3450 3300 60  0001 C CNN
 F 4 "0.00@0" H 3300 950 60  0001 C CNN "Pricing"
@@
 AR Path="/580A1257/5809B4E0" Ref="#PWR076"  Part="1"
 AR Path="/580A1261/5809B4E0" Ref="#PWR084"  Part="1"
-F 0 "#PWR084" H 3750 2400 50  0001 C CNN
+F 0 "#PWR060" H 3750 2400 50  0001 C CNN
 F 1 "GNDREF" H 3750 2500 50  0000 C CNN
 F 2 "" H 3750 2650 50  0000 C CNN
@@
 AR Path="/580A1257/5809B509" Ref="#PWR077"  Part="1"
 AR Path="/580A1261/5809B509" Ref="#PWR085"  Part="1"
-F 0 "#PWR085" H 2400 2200 50  0001 C CNN
+F 0 "#PWR061" H 2400 2200 50  0001 C CNN
 F 1 "GNDREF" H 2400 2300 50  0000 C CNN
 F 2 "" H 2400 2450 50  0000 C CNN
@@
 AR Path="/580A1257/5809B529" Ref="#PWR078"  Part="1"
 AR Path="/580A1261/5809B529" Ref="#PWR086"  Part="1"
-F 0 "#PWR086" H 2850 1450 50  0001 C CNN
+F 0 "#PWR062" H 2850 1450 50  0001 C CNN
 F 1 "GNDREF" H 2850 1550 50  0000 C CNN
 F 2 "" H 2850 1700 50  0000 C CNN
@@
 AR Path="/580A1257/5809B547" Ref="J8"  Part="1"
 AR Path="/580A1261/5809B547" Ref="J9"  Part="1"
-F 0 "J2" H 1800 1850 60  0000 C CNN
+F 0 "J6" H 1800 1850 60  0000 C CNN
 F 1 "JACK-TRS" H 1800 1950 60  0000 C CNN
-F 2 "" H 1800 1950 60  0000 C CNN
+F 2 "SW-KYCON:STX-3100-3C" H 1800 1950 60  0001 C CNN
 F 3 "" H 1800 1950 60  0000 C CNN
 	1    1800 1950
@@
 AR Path="/580A1257/5809B589" Ref="#PWR079"  Part="1"
 AR Path="/580A1261/5809B589" Ref="#PWR087"  Part="1"
-F 0 "#PWR087" H 4400 1600 50  0001 C CNN
+F 0 "#PWR063" H 4400 1600 50  0001 C CNN
 F 1 "+5VA" H 4400 1890 50  0000 C CNN
 F 2 "" H 4400 1750 50  0000 C CNN
@@
 AR Path="/580A1257/5809B5A3" Ref="#PWR080"  Part="1"
 AR Path="/580A1261/5809B5A3" Ref="#PWR088"  Part="1"
-F 0 "#PWR088" H 4050 1700 50  0001 C CNN
+F 0 "#PWR064" H 4050 1700 50  0001 C CNN
 F 1 "+5VD" H 4050 1990 50  0000 C CNN
 F 2 "" H 4050 1850 50  0000 C CNN
@@
 AR Path="/580A1257/5809B5C5" Ref="#PWR83"  Part="1"
 AR Path="/580A1261/5809B5C5" Ref="#PWR92"  Part="1"
-F 0 "#PWR29" H 2400 2250 50  0001 C CNN
+F 0 "#PWR65" H 2400 2250 50  0001 C CNN
 F 1 "-5V" H 2400 2300 50  0000 C CNN
 F 2 "" H 2400 2150 50  0000 C CNN
@@
 AR Path="/580A1257/5809B686" Ref="#PWR081"  Part="1"
 AR Path="/580A1261/5809B686" Ref="#PWR089"  Part="1"
-F 0 "#PWR089" H 2050 1400 50  0001 C CNN
+F 0 "#PWR065" H 2050 1400 50  0001 C CNN
 F 1 "GNDREF" H 2050 1500 50  0000 C CNN
 F 2 "" H 2050 1650 50  0000 C CNN
@@
 AR Path="/580A1257/5809B6F5" Ref="C37"  Part="1"
 AR Path="/580A1261/5809B6F5" Ref="C42"  Part="1"
-F 0 "C7" H 2525 2400 50  0000 L CNN
+F 0 "C27" H 2525 2400 50  0000 L CNN
 F 1 "0u01F" H 2525 2200 50  0000 L CNN
-F 2 "" H 2538 2150 50  0000 C CNN
+F 2 "Capacitors_SMD:C_0603_HandSoldering" H 2538 2150 50  0001 C CNN
 F 3 "" H 2500 2300 50  0000 C CNN
 	1    2500 2300
@@
 AR Path="/580A1257/5809B742" Ref="C40"  Part="1"
 AR Path="/580A1261/5809B742" Ref="C45"  Part="1"
-F 0 "C10" H 3825 1800 50  0000 L CNN
+F 0 "C30" H 3825 1800 50  0000 L CNN
 F 1 "0u01F" H 3825 1600 50  0000 L CNN
-F 2 "" H 3838 1550 50  0000 C CNN
+F 2 "Capacitors_SMD:C_0603_HandSoldering" H 3838 1550 50  0001 C CNN
 F 3 "" H 3800 1700 50  0000 C CNN
 	1    3800 1700
@@
 AR Path="/580A1257/5809B773" Ref="#PWR082"  Part="1"
 AR Path="/580A1261/5809B773" Ref="#PWR090"  Part="1"
-F 0 "#PWR090" H 3800 1300 50  0001 C CNN
+F 0 "#PWR066" H 3800 1300 50  0001 C CNN
 F 1 "GNDREF" H 3800 1400 50  0000 C CNN
 F 2 "" H 3800 1550 50  0000 C CNN
@@
 AR Path="/580A1257/5809B78A" Ref="C41"  Part="1"
 AR Path="/580A1261/5809B78A" Ref="C46"  Part="1"
-F 0 "C11" H 4575 1900 50  0000 L CNN
+F 0 "C31" H 4575 1900 50  0000 L CNN
 F 1 "0u01F" H 4575 1700 50  0000 L CNN
-F 2 "" H 4588 1650 50  0000 C CNN
+F 2 "Capacitors_SMD:C_0603_HandSoldering" H 4588 1650 50  0001 C CNN
 F 3 "" H 4550 1800 50  0000 C CNN
 	1    4550 1800
@@
 AR Path="/580A1257/5809B7BC" Ref="#PWR083"  Part="1"
 AR Path="/580A1261/5809B7BC" Ref="#PWR091"  Part="1"
-F 0 "#PWR091" H 4700 1550 50  0001 C CNN
+F 0 "#PWR067" H 4700 1550 50  0001 C CNN
 F 1 "GNDREF" H 4700 1650 50  0000 C CNN
 F 2 "" H 4700 1800 50  0000 C CNN
@@
 AR Path="/580A1257/580A32C0" Ref="R19"  Part="1"
 AR Path="/580A1261/580A32C0" Ref="R21"  Part="1"
-F 0 "R7" V 2230 2750 50  0000 C CNN
+F 0 "R15" V 2230 2750 50  0000 C CNN
 F 1 "10k" V 2150 2750 50  0000 C CNN
-F 2 "" V 2080 2750 50  0000 C CNN
+F 2 "Resistors_SMD:R_0805_HandSoldering" V 2080 2750 50  0001 C CNN
 F 3 "" H 2150 2750 50  0000 C CNN
 	1    2150 2750
@@
 AR Path="/580A1257/580A33C0" Ref="R20"  Part="1"
 AR Path="/580A1261/580A33C0" Ref="R22"  Part="1"
-F 0 "R8" V 2230 2950 50  0000 C CNN
+F 0 "R16" V 2230 2950 50  0000 C CNN
 F 1 "10k" V 2150 2950 50  0000 C CNN
-F 2 "" V 2080 2950 50  0000 C CNN
+F 2 "Resistors_SMD:R_0805_HandSoldering" V 2080 2950 50  0001 C CNN
 F 3 "" H 2150 2950 50  0000 C CNN
 	1    2150 2950
@@
 AR Path="/580A1257/580B5F27" Ref="C38"  Part="1"
 AR Path="/580A1261/580B5F27" Ref="C43"  Part="1"
-F 0 "C8" H 2575 2850 50  0000 L CNN
+F 0 "C28" H 2575 2850 50  0000 L CNN
 F 1 "1uF" H 2575 2650 50  0000 L CNN
-F 2 "" H 2588 2600 50  0000 C CNN
+F 2 "Capacitors_SMD:C_0603_HandSoldering" H 2588 2600 50  0001 C CNN
 F 3 "" H 2550 2750 50  0000 C CNN
 	1    2550 2750
@@
 AR Path="/580A1257/580B61C4" Ref="C39"  Part="1"
 AR Path="/580A1261/580B61C4" Ref="C44"  Part="1"
-F 0 "C9" H 2575 3050 50  0000 L CNN
+F 0 "C29" H 2575 3050 50  0000 L CNN
 F 1 "1uF" H 2575 2850 50  0000 L CNN
-F 2 "" H 2588 2800 50  0000 C CNN
+F 2 "Capacitors_SMD:C_0603_HandSoldering" H 2588 2800 50  0001 C CNN
 F 3 "" H 2550 2950 50  0000 C CNN
 	1    2550 2950

Commit message: replacing audio jack footprints
Parts:
- J2: footprint SW-KYCON:STX-3100-3C -> SW-CUI-INC:SJ1-353XNG-3Pin
Changed lines of the file:
@@
 AR Path="/580A1257/5809B3AA" Ref="U9"  Part="1"
 AR Path="/580A1261/5809B3AA" Ref="U10"  Part="1"
-F 0 "U7" V 3300 2400 60  0000 C CNN
+F 0 "U9" V 3300 2400 60  0000 C CNN
 F 1 "DS1882" V 3300 2000 60  0000 C CNN
 F 2 "Housings_SSOP:TSSOP-16_4.4x5mm_Pitch0.65mm" H 3200 2300 60  0001 C CNN
@@
 AR Path="/580A1257/5809B4E0" Ref="#PWR076"  Part="1"
 AR Path="/580A1261/5809B4E0" Ref="#PWR084"  Part="1"
-F 0 "#PWR060" H 3750 2400 50  0001 C CNN
+F 0 "#PWR076" H 3750 2400 50  0001 C CNN
 F 1 "GNDREF" H 3750 2500 50  0000 C CNN
 F 2 "" H 3750 2650 50  0000 C CNN
@@
 AR Path="/580A1257/5809B509" Ref="#PWR077"  Part="1"
 AR Path="/580A1261/5809B509" Ref="#PWR085"  Part="1"
-F 0 "#PWR061" H 2400 2200 50  0001 C CNN
+F 0 "#PWR077" H 2400 2200 50  0001 C CNN
 F 1 "GNDREF" H 2400 2300 50  0000 C CNN
 F 2 "" H 2400 2450 50  0000 C CNN
@@
 AR Path="/580A1257/5809B529" Ref="#PWR078"  Part="1"
 AR Path="/580A1261/5809B529" Ref="#PWR086"  Part="1"
-F 0 "#PWR062" H 2850 1450 50  0001 C CNN
+F 0 "#PWR078" H 2850 1450 50  0001 C CNN
 F 1 "GNDREF" H 2850 1550 50  0000 C CNN
 F 2 "" H 2850 1700 50  0000 C CNN
@@
 AR Path="/580A1257/5809B547" Ref="J8"  Part="1"
 AR Path="/580A1261/5809B547" Ref="J9"  Part="1"
-F 0 "J6" H 1800 1850 60  0000 C CNN
+F 0 "J8" H 1800 1850 60  0000 C CNN
 F 1 "JACK-TRS" H 1800 1950 60  0000 C CNN
-F 2 "SW-KYCON:STX-3100-3C" H 1800 1950 60  0001 C CNN
+F 2 "SW-CUI-INC:SJ1-353XNG-3Pin" H 1800 1950 60  0001 C CNN
 F 3 "" H 1800 1950 60  0000 C CNN
 	1    1800 1950
@@
 AR Path="/580A1257/5809B589" Ref="#PWR079"  Part="1"
 AR Path="/580A1261/5809B589" Ref="#PWR087"  Part="1"
-F 0 "#PWR063" H 4400 1600 50  0001 C CNN
+F 0 "#PWR079" H 4400 1600 50  0001 C CNN
 F 1 "+5VA" H 4400 1890 50  0000 C CNN
 F 2 "" H 4400 1750 50  0000 C CNN
@@
 AR Path="/580A1257/5809B5A3" Ref="#PWR080"  Part="1"
 AR Path="/580A1261/5809B5A3" Ref="#PWR088"  Part="1"
-F 0 "#PWR064" H 4050 1700 50  0001 C CNN
+F 0 "#PWR080" H 4050 1700 50  0001 C CNN
 F 1 "+5VD" H 4050 1990 50  0000 C CNN
 F 2 "" H 4050 1850 50  0000 C CNN
@@
 AR Path="/580A1257/5809B5C5" Ref="#PWR83"  Part="1"
 AR Path="/580A1261/5809B5C5" Ref="#PWR92"  Part="1"
-F 0 "#PWR65" H 2400 2250 50  0001 C CNN
+F 0 "#PWR83" H 2400 2250 50  0001 C CNN
 F 1 "-5V" H 2400 2300 50  0000 C CNN
 F 2 "" H 2400 2150 50  0000 C CNN
@@
 AR Path="/580A1257/5809B686" Ref="#PWR081"  Part="1"
 AR Path="/580A1261/5809B686" Ref="#PWR089"  Part="1"
-F 0 "#PWR065" H 2050 1400 50  0001 C CNN
+F 0 "#PWR081" H 2050 1400 50  0001 C CNN
 F 1 "GNDREF" H 2050 1500 50  0000 C CNN
 F 2 "" H 2050 1650 50  0000 C CNN
@@
 AR Path="/580A1257/5809B6F5" Ref="C37"  Part="1"
 AR Path="/580A1261/5809B6F5" Ref="C42"  Part="1"
-F 0 "C27" H 2525 2400 50  0000 L CNN
+F 0 "C37" H 2525 2400 50  0000 L CNN
 F 1 "0u01F" H 2525 2200 50  0000 L CNN
 F 2 "Capacitors_SMD:C_0603_HandSoldering" H 2538 2150 50  0001 C CNN
@@
 AR Path="/580A1257/5809B742" Ref="C40"  Part="1"
 AR Path="/580A1261/5809B742" Ref="C45"  Part="1"
-F 0 "C30" H 3825 1800 50  0000 L CNN
+F 0 "C40" H 3825 1800 50  0000 L CNN
 F 1 "0u01F" H 3825 1600 50  0000 L CNN
 F 2 "Capacitors_SMD:C_0603_HandSoldering" H 3838 1550 50  0001 C CNN
@@
 AR Path="/580A1257/5809B773" Ref="#PWR082"  Part="1"
 AR Path="/580A1261/5809B773" Ref="#PWR090"  Part="1"
-F 0 "#PWR066" H 3800 1300 50  0001 C CNN
+F 0 "#PWR082" H 3800 1300 50  0001 C CNN
 F 1 "GNDREF" H 3800 1400 50  0000 C CNN
 F 2 "" H 3800 1550 50  0000 C CNN
@@
 AR Path="/580A1257/5809B78A" Ref="C41"  Part="1"
 AR Path="/580A1261/5809B78A" Ref="C46"  Part="1"
-F 0 "C31" H 4575 1900 50  0000 L CNN
+F 0 "C41" H 4575 1900 50  0000 L CNN
 F 1 "0u01F" H 4575 1700 50  0000 L CNN
 F 2 "Capacitors_SMD:C_0603_HandSoldering" H 4588 1650 50  0001 C CNN
@@
 AR Path="/580A1257/5809B7BC" Ref="#PWR083"  Part="1"
 AR Path="/580A1261/5809B7BC" Ref="#PWR091"  Part="1"
-F 0 "#PWR067" H 4700 1550 50  0001 C CNN
+F 0 "#PWR083" H 4700 1550 50  0001 C CNN
 F 1 "GNDREF" H 4700 1650 50  0000 C CNN
 F 2 "" H 4700 1800 50  0000 C CNN
@@
 AR Path="/580A1257/580A32C0" Ref="R19"  Part="1"
 AR Path="/580A1261/580A32C0" Ref="R21"  Part="1"
-F 0 "R15" V 2230 2750 50  0000 C CNN
+F 0 "R19" V 2230 2750 50  0000 C CNN
 F 1 "10k" V 2150 2750 50  0000 C CNN
 F 2 "Resistors_SMD:R_0805_HandSoldering" V 2080 2750 50  0001 C CNN
@@
 AR Path="/580A1257/580A33C0" Ref="R20"  Part="1"
 AR Path="/580A1261/580A33C0" Ref="R22"  Part="1"
-F 0 "R16" V 2230 2950 50  0000 C CNN
+F 0 "R20" V 2230 2950 50  0000 C CNN
 F 1 "10k" V 2150 2950 50  0000 C CNN
 F 2 "Resistors_SMD:R_0805_HandSoldering" V 2080 2950 50  0001 C CNN
@@
 AR Path="/580A1257/580B5F27" Ref="C38"  Part="1"
 AR Path="/580A1261/580B5F27" Ref="C43"  Part="1"
-F 0 "C28" H 2575 2850 50  0000 L CNN
+F 0 "C38" H 2575 2850 50  0000 L CNN
 F 1 "1uF" H 2575 2650 50  0000 L CNN
 F 2 "Capacitors_SMD:C_0603_HandSoldering" H 2588 2600 50  0001 C CNN
@@
 AR Path="/580A1257/580B61C4" Ref="C39"  Part="1"
 AR Path="/580A1261/580B61C4" Ref="C44"  Part="1"
-F 0 "C29" H 2575 3050 50  0000 L CNN
+F 0 "C39" H 2575 3050 50  0000 L CNN
 F 1 "1uF" H 2575 2850 50  0000 L CNN
 F 2 "Capacitors_SMD:C_0603_HandSoldering" H 2588 2800 50  0001 C CNN
