File: portable-line-mixer.kicad_pcb (KiCad board)
At the start: 2 copper layers, 155 parts, among them CON1 BARREL_JACK, J1 JACK-TRS, J2 JACK-TRS, J3 JACK-TRS, J4 JACK-TRS, J5 JACK-TRS, J6 JACK-TRS, J7 JACK-TRS, J8 JACK-TRS, J9 JACK-TRS, P1 USB_OTG, SW1 RESET, SW3 ON/OFF, T1 PMV45EN2, T2 PMV45EN2, T3 PMV45EN2, T4 PMV45EN2, T5 PMV48XP, U1 RC4560, U10 DS1882, U11 LT1085, U12 NCP1117ST50T3G_MountingTab, U13 MAX1721, U14 NCP1117ST50T3G_MountingTab, U15 MAX6820, U16 NCP1117ST50T3G_MountingTab, U17 MAX6820, U18 LT3580, U19 ATMEGA32U4-A, U2 RC4560, U3 DS1882, U4 DS1882, U5 DS1882, U6 DS1882, U7 DS1882, U8 DS1882, U9 DS1882, Y1 LFXTAL056036

Commit message: replacing audio jack footprints
Parts:
- J1, J2, J3, J4, J5, J6, J7, J8, J9: footprint SW-KYCON:STX-3100-3C -> SW-CUI-INC:SJ1-353XNG-3Pin

Commit message: before initial DRC
Parts:
- added R34: 4k7, Capacitors_SMD:C_0805_HandSoldering, B.Cu at (158.1, 112.4)
- added R35: 4k7, Capacitors_SMD:C_0805_HandSoldering, B.Cu at (154.9, 111.1)
- C55, C59: value 40mF -> 0u01F
- moved C69 99.6 mm to (129.8, 81.5), turned to 0 degrees
- moved R33 99.1 mm to (125.2, 86.6), turned to 270 degrees
- moved C72 95.7 mm to (129.5, 84.3), turned to 0 degrees
- moved D2 94.0 mm to (122.2, 86.6), turned to 270 degrees
- moved C70 93.5 mm to (129.5, 86.1), turned to 0 degrees
- moved C71 91.9 mm to (129.5, 87.9), turned to 0 degrees
- moved F1 90.8 mm to (124.2, 103.4)
- moved L1 89.1 mm to (116.1, 36.3), turned to 90 degrees
- moved C61 83.5 mm to (108.7, 44.7), turned to 270 degrees
- moved C66 82.9 mm to (129.3, 106.4), turned to 270 degrees
- moved C64 81.1 mm to (113.5, 49.5), turned to 180 degrees
- moved C65 79.0 mm to (124.3, 108.0)
- moved R31 79.0 mm to (131.1, 106.7), turned to 90 degrees
- moved C58 79.0 mm to (102.1, 39.4), turned to 270 degrees
- moved T3 78.6 mm to (125.5, 42.9)
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Connections:
- net Net-(D2-Pad2) renamed /Microprocessor/RESET
- net Net-(P1-Pad2) renamed /Microprocessor/D-
- net Net-(P1-Pad3) renamed /Microprocessor/D+
- net Net-(R30-Pad1) renamed /Microprocessor/USB-D+
- net Net-(R32-Pad1) renamed /Microprocessor/USB-D-
- net Net-(S1-Pad1) renamed /Microprocessor/ENC-1
- net Net-(S1-Pad3) renamed /Microprocessor/ENC-A
- net Net-(S1-Pad5) renamed /Microprocessor/ENC-B
- U19 pad 30: Net-(U19-Pad30) -> GNDREF
Routing:
- net GNDREF: track 0.00 -> 374.1 mm, vias 0 -> 36
- net +5VD: track 0.00 -> 169.2 mm, vias 0 -> 11
- net +5VA: track 0.00 -> 158.0 mm, vias 0 -> 13
- net -5V: track 0.00 -> 150.7 mm, vias 0 -> 9
- net /SDA: track 0.00 -> 130.3 mm, vias 0 -> 9
- net /SCL: track 0.00 -> 126.2 mm, vias 0 -> 9
- net /~CE: track 0.00 -> 122.7 mm, vias 0 -> 11
- net Net-(C48-Pad1): track 0.00 -> 116.8 mm, vias 0 -> 8
- net +5VP: track 0.00 -> 106.4 mm, vias 0 -> 3
- net /Microprocessor/+5VARD: track 0.00 -> 90.2 mm
- net /Stereo-Input-0/LOUT: track 0.00 -> 85.1 mm, vias 0 -> 2
- net /Stereo-Input-0/ROUT: track 0.00 -> 83.0 mm, vias 0 -> 2
- net /Microprocessor/ENC-A: track 0.00 -> 49.6 mm, vias 0 -> 1
- net /Microprocessor/ENC-B: track 0.00 -> 43.3 mm, vias 0 -> 1
- net Net-(C57-Pad1): track 0.00 -> 42.8 mm
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- added copper zone on B.Cu, net GNDREF
- added copper zone on F.Cu, net GNDREF
Other:
- board outline added: 97.8 x 83.8 mm
- net class Default: clearance 0.2 -> 0.1524; trace_width 0.25 -> 0.1524; via_dia 0.6 -> 0.6858; via_drill 0.4 -> 0.3302
- rule trace_clearance: 0.2 -> 0.1524
- rule trace_min: 0.2 -> 0.1524
- rule via_min_drill: 0.3 -> 0.3302
- rule via_min_size: 0.4 -> 0.6858

Commit message: after DRC and fixes
Routing:
- net /Stereo-Input-0/ROUT: track 83.0 -> 91.9 mm
- net GNDREF: track 374.1 -> 382.1 mm, vias 36 -> 38
- net Net-(C23-Pad2): track 0.00 -> 3.41 mm
