File: portable-line-mixer.kicad_pcb (KiCad board)
At the start: 4 copper layers, 142.2 x 209.6 mm, 138 parts, among them J1 Power In (Male-top), J2 LCD Connection I2C, J3 Audio Out, J4 Audio IN, SW1 Nano Reset, U1 LM27762, U10 DS1882, U11 DS1882, U12 DS1882, U13 DS1882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

Commit message: Swapped encoder for connector
Parts:
- removed S1: PEC11-4215F-S24, SW-Bournes:PEC11R-4xxx-Sxxxx
- added J5: Encoder Connection, SW-Hirose:DF11-4DP-2DSA, F.Cu at (193.7, 261.0)
- added T1: PMV45EN2, Package_TO_SOT_SMD:SOT-23, F.Cu at (165.9, 246.8)
- U1: footprint Package_SON:WSON-12-1EP_3x2mm_P0.5mm -> SW-Package-SON:WSON-12-1EP_3x2mm_P0.5mm
- moved C4 88.4 mm to (162.5, 248.3), turned to 90 degrees
- moved C5 87.7 mm to (160.1, 248.3), turned to 90 degrees
- moved R2 85.6 mm to (164.6, 250.7), turned to 270 degrees
- moved C3 83.0 mm to (156.6, 250.7), turned to 90 degrees
- moved U1 82.6 mm to (161.8, 252.4), turned to 270 degrees
- moved R1 82.3 mm to (165.4, 253.2), turned to 0 degrees
- moved R6 80.3 mm to (158.6, 253.2), turned to 270 degrees
- moved C1 78.7 mm to (165.7, 256.7), turned to 270 degrees
- moved R7 78.6 mm to (156.0, 254.3), turned to 180 degrees
- moved C2 78.4 mm to (161.9, 255.3), turned to 180 degrees
Routing:
- net GNDREF: track 16.6 -> 0.00 mm, vias 137 -> 130
- net -5VA: track 47.0 -> 33.5 mm
- net +5VA: track 44.4 -> 36.8 mm
- net Net-(R1-Pad2): track 0.00 -> 7.27 mm
- net Net-(R10-Pad2): track 6.99 -> 0.00 mm
- net /Power Handling/±5VA_EN: track 1.57 -> 6.44 mm
- net +5V: track 2.07 -> 5.04 mm, vias 62 -> 61
- net Net-(C2-Pad2): track 2.35 -> 2.91 mm
Other:
- board text added: "Mount Connectors at top of pcb Mount LCD screen facing up parallel to pcb Use clear plastic for lid of enclosure Mount Encoder at bottom of pcb and build protective shrouding around knob"

Commit message: Portable Line Mixer done
Parts:
- removed MK4: Mounting_Hole_PAD, MountingHole:MountingHole_4.3mm_M4_Pad_Via
- MK1, MK2, MK3: footprint MountingHole:MountingHole_4.3mm_M4_Pad_Via -> MountingHole:MountingHole_2.7mm_M2.5_Pad_Via
- U5: footprint Package_SSOP:HTSSOP-20-1EP_4.4x6.5mm_P0.65mm_EP3.4x6.5mm_ThermalVias -> SW-Linear:TSSOP-20-1EP_4.4x6.5mm_P0.65mm_EP2.75x6.07mm-LTC3265
- moved J1 262.8 mm to (74.2, 139.1), turned to 180 degrees
- moved F1 254.9 mm to (69.2, 145.4), turned to 270 degrees
- moved C6 231.1 mm to (72.1, 152.9), turned to 0 degrees
- moved U3 213.6 mm to (73.2, 163.9), turned to 270 degrees
- moved C7 198.2 mm to (74.6, 173.7), turned to 0 degrees
- moved R8 194.7 mm to (75.1, 175.7), turned to 180 degrees
- moved R11 190.9 mm to (69.8, 117.1), turned to 90 degrees
- moved C15 184.9 mm to (71.8, 117.0), turned to 90 degrees
- moved C11 180.6 mm to (77.9, 124.6)
- moved C16 175.9 mm to (78.4, 132.8), turned to 0 degrees
- moved C13 174.9 mm to (69.6, 133.5), turned to 0 degrees
- moved C10 170.0 mm to (67.9, 127.9), turned to 90 degrees
- moved SW1 162.0 mm to (135.9, 102.9), turned to 90 degrees
- moved C20 151.8 mm to (80.0, 107.5), turned to 270 degrees
- moved C12 151.2 mm to (67.8, 116.3), turned to 270 degrees
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Connections:
- net Net-(C10-Pad1) renamed /Power Handling/CBST-
- net Net-(C10-Pad2) renamed /Power Handling/CBST+
- net Net-(C11-Pad1) renamed /Power Handling/CINV-
- net Net-(C11-Pad2) renamed /Power Handling/CINV+
- net Net-(C14-Pad2) renamed /Power Handling/BYP-
- net Net-(C15-Pad1) renamed /Power Handling/BYP+
- net Net-(C17-Pad2) renamed /Power Handling/VOUT+
- net Net-(C18-Pad2) renamed /Power Handling/VOUT-
- net Net-(R10-Pad2) renamed /Power Handling/ADJ+
- net Net-(R12-Pad2) renamed /Power Handling/ADJ-
- J2 pad 1: /Arduino Nano Header Connections + Ethernet connection/5V-SCL -> +5V
- J2 pad 2: +5V -> GNDREF
- J2 pad 3: /Arduino Nano Header Connections + Ethernet connection/5V-SDA -> /Arduino Nano Header Connections + Ethernet connection/5V-SCL
- J2 pad 4: GNDREF -> /Arduino Nano Header Connections + Ethernet connection/5V-SDA
- J5 pad 1: GNDREF -> /Arduino Nano Header Connections + Ethernet connection/ENC-1
- J5 pad 2: /Arduino Nano Header Connections + Ethernet connection/ENC-B -> GNDREF
- J5 pad 3: /Arduino Nano Header Connections + Ethernet connection/ENC-1 -> /Arduino Nano Header Connections + Ethernet connection/ENC-A
- J5 pad 4: /Arduino Nano Header Connections + Ethernet connection/ENC-A -> /Arduino Nano Header Connections + Ethernet connection/ENC-B
Routing:
- net /Power Handling/±12VA_EN: track 0.00 -> 117.3 mm, vias 0 -> 3
- net /Arduino Nano Header Connections + Ethernet connection/5V-SCL: track 0.00 -> 111.4 mm, vias 1 -> 8
- net /Arduino Nano Header Connections + Ethernet connection/5V-SDA: track 0.00 -> 104.3 mm, vias 0 -> 9
- net /Arduino Nano Header Connections + Ethernet connection/Nano_RST: track 0.00 -> 101.5 mm
- net /Audio Mixer/L-IN0: track 2.43 -> 97.6 mm, vias 1 -> 0
- net /Audio Mixer/L-IN1: track 2.44 -> 94.5 mm, vias 1 -> 0
- net /Audio Mixer/R-IN0: track 2.46 -> 93.3 mm, vias 1 -> 0
- net /Audio Mixer/R-IN1: track 2.44 -> 90.2 mm, vias 1 -> 0
- net /Audio Mixer/L-IN2: track 2.47 -> 81.7 mm, vias 1 -> 0
- net /Audio Mixer/R-IN2: track 2.42 -> 78.6 mm, vias 1 -> 0
- net /Audio Mixer/L-IN3: track 2.43 -> 78.2 mm
- net /Audio Mixer/R-IN3: track 2.46 -> 74.6 mm
- net /Audio Mixer/R_MIX_BUS: track 78.8 -> 149.4 mm, vias 8 -> 9
- net /Audio Mixer/L-IN4: track 2.51 -> 65.8 mm
- net /Audio Mixer/L-IN5: track 2.47 -> 63.2 mm, vias 1 -> 0
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- added copper zone on In1.Cu, net +12V
- added copper zone on B.Cu, net +5V
- added copper zone on In1.Cu, net +5V
- added copper zone on B.Cu, net GNDREF
- added copper zone on F.Cu, net Net-(R22-Pad1)
Other:
- board size 142.2 x 209.6 mm -> 77.5 x 114.3 mm
- board text removed: "HDST-0"
