File: microprocessor.sch (KiCad schematic (older format))
At the start: 26 parts

Commit message: finished with first draft of schematic
Parts:
- gave numbers to parts that had none: 26
Connections:
- net GNDREF: now also P1.6 (shield), S1.2 (S2), S1.4 (C)
- net at R33.2, SW1.2, U19.13 (~RESET~): now also D2.2 (A)
- net at U19.1 ((INT6/AIN0)PE6): now also S1.1 (S1)
- net at U19.20 ((RXD/INT2)PD2): now also S1.5 (B)
- net TXserial: now reaches U19.21 ((TXD/INT3)PD3)
- net at U19.27 ((T0/OC4D/ADC10)PD7): now also S1.3 (A)
- net +5VD renamed +5VP
- no-connect marks 1 -> 20
Other:
- note added: "This p type MOSFET will connect VUSB to D\nif there is no power from +5VP which is tied to ground"
- note added: "Use D0(PD2) and D7(PE6) as interupts for encoder,\n1 for detecting switch and one for\ndetecting transition which is less \nimportant so only 1/2 accuacy is acceptable.\nOther encoder pin is connected to D6(PD7)\nMake certain to turn on pullup resistors on\nthese pins as they will be pulled low on\nchange."
- note added: "tx serial is used for \npotential serial LCD \ndisplay"
- note removed: "This p type MOSFET will connect VUSB to D\nif there is no power from +5VD which is tied to ground"
- moved on the sheet: S1

Commit message: finalized schematic, finishing footprint assignment, starting pcb layout
Parts:
- removed C65: 22uF, symbol C_Small
- added C65: 22uF, Capacitors_Tantalum_SMD:TantalC_SizeB_EIA-3528_HandSoldering, symbol CP_Small
- C66, C67, C68, C70, C71, C72, C73, C74, C75, Z1, Z2: footprint (none) -> Capacitors_SMD:C_0603_HandSoldering
- C69: footprint (none) -> Capacitors_Tantalum_SMD:TantalC_SizeB_EIA-3528_HandSoldering
- D2: footprint (none) -> Capacitors_SMD:C_1206_HandSoldering
- F1: footprint (none) -> Capacitors_SMD:C_1812_HandSoldering
- L3, R30, R31, R32, R33: footprint (none) -> Resistors_SMD:R_0805_HandSoldering
- P1: footprint (none) -> SW-Hirose:ZX62D-B-5PA8(30)
- S1: footprint (none) -> SW-Bournes:PEC11R-4xxx-Sxxxx
- SW1: footprint (none) -> SW-Eswitch:M7
- T5: renamed from T1; footprint SOT23 -> TO_SOT_Packages_SMD:SOT-23
- U19: footprint TQFP44 -> Housings_QFP:TQFP-44_10x10mm_Pitch0.8mm
- Y1: footprint (none) -> SW-IQD:CFPX-180
Connections:
- net GNDREF: now also C65.2
- net at C67.2, Y1.3 (Crystal): now also U19.16 (XTAL2); no longer U19.17 (XTAL1)
- net at C68.1, Y1.1 (Crystal): now also U19.17 (XTAL1); no longer U19.16 (XTAL2)
- net at F1.2, P1.1 (VCC): now also C65.1
Changed lines of the file:
@@
 F 0 "U19" H 4850 5600 50  0000 C CNN
 F 1 "ATMEGA32U4-A" H 6500 2400 50  0000 C CNN
-F 2 "TQFP44" H 5800 3900 50  0000 C CIN
+F 2 "Housings_QFP:TQFP-44_10x10mm_Pitch0.8mm" H 5800 3900 50  0000 C CIN
 F 3 "" H 6900 5000 50  0000 C CNN
 	1    5800 3900
@@
 F 0 "S1" H 8250 3950 60  0000 C CNN
 F 1 "PEC11-4215F-S24" H 8250 3600 60  0000 C CNN
-F 2 "" H 8150 3850 60  0001 C CNN
+F 2 "SW-Bournes:PEC11R-4xxx-Sxxxx" H 8150 3850 60  0001 C CNN
 F 3 "http://www.bourns.com/docs/Product-Datasheets/pec11R.pdf" H 8100 4150 60  0001 C CNN
 F 4 "0.00@0" H 8550 4450 60  0001 C CNN "Pricing"
@@
 F 0 "P1" H 3075 3575 50  0000 C CNN
 F 1 "USB_OTG" H 2750 3900 50  0000 C CNN
-F 2 "" V 2700 3600 50  0000 C CNN
+F 2 "SW-Hirose:ZX62D-B-5PA8(30)" V 2700 3600 50  0001 C CNN
 F 3 "" V 2700 3600 50  0000 C CNN
 	1    2750 3700
@@
 $EndComp
 $Comp
-L MF-MSMF050-2 F1
-U 1 1 580C7F4B
-P 3400 4000
-F 0 "F1" H 3400 4000 60  0000 C CNN
-F 1 "MF-MSMF050-2" H 3400 3900 60  0000 C CNN
-F 2 "" H 3300 3900 60  0001 C CNN
-F 3 "https://www.bourns.com/PDFs/MFMSMF.pdf" H 3350 3700 60  0001 C CNN
-F 4 "0.00@0" H 3600 3800 60  0001 C CNN "Pricing"
-F 5 "1812 mils" H 3400 4400 60  0001 C CNN "Package ID"
-F 6 "Bournes" H 3400 4200 60  0001 C CNN "Manufacturer"
-F 7 "PTC Resettable Fuses" H 3400 4300 60  0001 C CNN "Description"
-	1    3400 4000
-	1    0    0    -1
-$EndComp
-$Comp
-L PMV48XP T1
+L PMV48XP T5
 U 1 1 580C85DC
 P 5250 1500
-F 0 "T1" H 5500 1575 50  0000 L CNN
+F 0 "T5" H 5500 1575 50  0000 L CNN
 F 1 "PMV48XP" H 5500 1500 50  0000 L CNN
-F 2 "SOT23" H 5500 1400 50  0001 L CIN
+F 2 "TO_SOT_Packages_SMD:SOT-23" H 5500 1400 50  0001 L CIN
 F 3 "http://www.nxp.com/documents/data_sheet/PMV48XP.pdf" H 4900 2150 50  0001 L CNN
 F 4 "0.00@0" H 5250 1100 60  0001 C CNN "Pricing"
@@
 F 0 "D2" H 4450 2100 50  0000 C CNN
 F 1 "CD1206-S01575" H 4450 2300 50  0000 C CNN
-F 2 "" H 4450 2200 50  0000 C CNN
+F 2 "Capacitors_SMD:C_1206_HandSoldering" H 4450 2200 50  0001 C CNN
 F 3 "" H 4450 2200 50  0000 C CNN
 	1    4450 2200
@@
 F 0 "Y1" H 3800 2850 60  0000 C CNN
 F 1 "LFXTAL056036" H 3850 2600 60  0000 C CNN
-F 2 "" H 3800 3000 60  0001 C CNN
+F 2 "SW-IQD:CFPX-180" H 3800 3000 60  0001 C CNN
 F 3 "http://www.mouser.com/ds/2/741/LFXTAL056036Reel-999733.pdf" H 3850 2550 60  0001 C CNN
 F 4 "0.00@0" H 3600 3400 60  0001 C CNN "Pricing"
@@
 F 0 "R32" V 4030 3800 50  0000 C CNN
 F 1 "22R" V 3950 3800 50  0000 C CNN
-F 2 "" V 3880 3800 50  0000 C CNN
+F 2 "Resistors_SMD:R_0805_HandSoldering" V 3880 3800 50  0001 C CNN
 F 3 "" H 3950 3800 50  0000 C CNN
 	1    3950 3800
@@
 F 0 "R30" V 3730 3700 50  0000 C CNN
 F 1 "22R" V 3650 3700 50  0000 C CNN
-F 2 "" V 3580 3700 50  0000 C CNN
+F 2 "Resistors_SMD:R_0805_HandSoldering" V 3580 3700 50  0001 C CNN
 F 3 "" H 3650 3700 50  0000 C CNN
 	1    3650 3700
@@
 F 0 "Z1" H 3200 3500 60  0000 C CNN
 F 1 "CG0603MLC-05E" H 3200 3600 60  0000 C CNN
-F 2 "" H 3100 3400 60  0001 C CNN
+F 2 "Capacitors_SMD:C_0603_HandSoldering" H 3100 3400 60  0001 C CNN
 F 3 "http://bourns.com/pdfs/MLC.pdf" H 3150 3200 60  0001 C CNN
 F 4 "0.00@0" H 3400 3300 60  0001 C CNN "Pricing"
@@
 F 0 "Z2" H 3400 3300 60  0000 C CNN
 F 1 "CG0603MLC-05E" H 3400 3400 60  0000 C CNN
-F 2 "" H 3300 3200 60  0001 C CNN
+F 2 "Capacitors_SMD:C_0603_HandSoldering" H 3300 3200 60  0001 C CNN
 F 3 "http://bourns.com/pdfs/MLC.pdf" H 3350 3000 60  0001 C CNN
 F 4 "0.00@0" H 3600 3100 60  0001 C CNN "Pricing"
@@
 F 0 "C67" H 4160 2620 50  0000 L CNN
 F 1 "22pF" H 4160 2470 50  0000 L CNN
-F 2 "" H 4150 2550 50  0000 C CNN
+F 2 "Capacitors_SMD:C_0603_HandSoldering" H 4150 2550 50  0001 C CNN
 F 3 "" H 4150 2550 50  0000 C CNN
 	1    4150 2550
@@
 F 0 "C68" H 4160 3220 50  0000 L CNN
 F 1 "22pF" H 4160 3070 50  0000 L CNN
-F 2 "" H 4150 3150 50  0000 C CNN
+F 2 "Capacitors_SMD:C_0603_HandSoldering" H 4150 3150 50  0001 C CNN
 F 3 "" H 4150 3150 50  0000 C CNN
 	1    4150 3150
@@
 Connection ~ 3200 3700
 Wire Wire Line
-	4150 2750 4650 2750
-Wire Wire Line
-	4650 2950 4150 2950
-Wire Wire Line
 	4150 2650 4150 2750
 Wire Wire Line
 	4150 2950 4150 3050
 Wire Wire Line
-	3450 3100 3450 2450
+	3450 2450 3450 3100
 Wire Wire Line
 	4150 3250 3600 3250
@@
 Connection ~ 3400 3100
 Wire Wire Line
-	3050 3500 3050 3000
+	3050 3000 3050 3500
 Wire Wire Line
 	3050 3000 3200 3000
@@
 F 0 "C74" H 4560 4970 50  0000 L CNN
 F 1 "100nF" H 4560 4820 50  0000 L CNN
-F 2 "" H 4550 4900 50  0000 C CNN
+F 2 "Capacitors_SMD:C_0603_HandSoldering" H 4550 4900 50  0001 C CNN
 F 3 "" H 4550 4900 50  0000 C CNN
 	1    4550 4900
@@
 F 0 "C73" H 4560 4220 50  0000 L CNN
 F 1 "1uF" H 4560 4070 50  0000 L CNN
-F 2 "" H 4550 4150 50  0000 C CNN
+F 2 "Capacitors_SMD:C_0603_HandSoldering" H 4550 4150 50  0001 C CNN
 F 3 "" H 4550 4150 50  0000 C CNN
 	1    4550 4150
@@
 Text Label 3950 4000 0    60   ~ 0
 VUSB
-$Comp
-L C_Small C65
-U 1 1 580AD2E6
-P 3050 4350
-F 0 "C65" H 3060 4420 50  0000 L CNN
-F 1 "22uF" H 3060 4270 50  0000 L CNN
-F 2 "" H 3050 4350 50  0000 C CNN
-F 3 "" H 3050 4350 50  0000 C CNN
-	1    3050 4350
-	1    0    0    -1
-$EndComp
 Wire Wire Line
 	3200 4000 3050 4000
@@
 F 0 "R31" V 3780 4300 50  0000 C CNN
 F 1 "22R" V 3700 4300 50  0000 C CNN
-F 2 "" V 3630 4300 50  0000 C CNN
+F 2 "Resistors_SMD:R_0805_HandSoldering" V 3630 4300 50  0001 C CNN
 F 3 "" H 3700 4300 50  0000 C CNN
 	1    3700 4300
@@
 F 0 "C66" H 3860 4420 50  0000 L CNN
 F 1 "100nF" H 3860 4270 50  0000 L CNN
-F 2 "" H 3850 4350 50  0000 C CNN
+F 2 "Capacitors_SMD:C_0603_HandSoldering" H 3850 4350 50  0001 C CNN
 F 3 "" H 3850 4350 50  0000 C CNN
 	1    3850 4350
@@
 F 0 "L3" H 6050 1950 60  0000 C CNN
 F 1 "MH2029-300Y" H 6050 1750 60  0000 C CNN
-F 2 "" H 5950 1850 60  0001 C CNN
+F 2 "Resistors_SMD:R_0805_HandSoldering" H 5950 1850 60  0001 C CNN
 F 3 "http://www.mouser.com/ds/2/54/h-777565.pdf" H 6200 2000 60  0001 C CNN
 F 4 "0.00@0" H 5800 2100 60  0001 C CNN "Pricing"
@@
 F 0 "C75" H 6360 2120 50  0000 L CNN
 F 1 "1uF" H 6360 1970 50  0000 L CNN
-F 2 "" H 6350 2050 50  0000 C CNN
+F 2 "Capacitors_SMD:C_0603_HandSoldering" H 6350 2050 50  0001 C CNN
 F 3 "" H 6350 2050 50  0000 C CNN
 	1    6350 2050
@@
 F 0 "SW1" H 4100 2450 50  0000 C CNN
 F 1 "RESET" H 4250 2300 50  0000 C CNN
-F 2 "" H 4250 2550 50  0000 C CNN
+F 2 "SW-Eswitch:M7" H 4250 2550 50  0001 C CNN
 F 3 "" H 4250 2550 50  0000 C CNN
 	1    4250 2350
@@
 F 0 "R33" V 4730 2200 50  0000 C CNN
 F 1 "10k" V 4650 2200 50  0000 C CNN
-F 2 "" V 4580 2200 50  0000 C CNN
+F 2 "Resistors_SMD:R_0805_HandSoldering" V 4580 2200 50  0001 C CNN
 F 3 "" H 4650 2200 50  0000 C CNN
 	1    4650 2200
@@
 F 0 "C72" H 4360 1870 50  0000 L CNN
 F 1 "100nF" H 4360 1720 50  0000 L CNN
-F 2 "" H 4350 1800 50  0000 C CNN
+F 2 "Capacitors_SMD:C_0603_HandSoldering" H 4350 1800 50  0001 C CNN
 F 3 "" H 4350 1800 50  0000 C CNN
 	1    4350 1800
@@
 F 0 "C71" H 4360 1620 50  0000 L CNN
 F 1 "100nF" V 4250 1450 50  0000 L CNN
-F 2 "" H 4350 1550 50  0000 C CNN
+F 2 "Capacitors_SMD:C_0603_HandSoldering" H 4350 1550 50  0001 C CNN
 F 3 "" H 4350 1550 50  0000 C CNN
 	1    4350 1550
@@
 F 0 "C70" H 4360 1420 50  0000 L CNN
 F 1 "100nF" V 4250 1250 50  0000 L CNN
-F 2 "" H 4350 1350 50  0000 C CNN
+F 2 "Capacitors_SMD:C_0603_HandSoldering" H 4350 1350 50  0001 C CNN
 F 3 "" H 4350 1350 50  0000 C CNN
 	1    4350 1350
@@
 F 0 "C69" H 4360 1170 50  0000 L CNN
 F 1 "22uF" V 4250 1050 50  0000 L CNN
-F 2 "" H 4350 1100 50  0000 C CNN
+F 2 "Capacitors_Tantalum_SMD:TantalC_SizeB_EIA-3528_HandSoldering" H 4350 1100 50  0001 C CNN
 F 3 "" H 4350 1100 50  0000 C CNN
 	1    4350 1100
@@
 	1    0    0    -1
 $EndComp
+$Comp
+L CP_Small C65
+U 1 1 5813C5FE
+P 3050 4350
+F 0 "C65" H 3060 4420 50  0000 L CNN
+F 1 "22uF" H 3060 4270 50  0000 L CNN
+F 2 "Capacitors_Tantalum_SMD:TantalC_SizeB_EIA-3528_HandSoldering" H 3050 4350 50  0001 C CNN
+F 3 "" H 3050 4350 50  0000 C CNN
+	1    3050 4350
+	1    0    0    -1
+$EndComp
+Text Notes 2250 4700 0    60   ~ 0
+Polar Tantalum\ncapacitor\nwith solid \nelectrolyte
+$Comp
+L MF-MSMF050-2 F1
+U 1 1 58142C3D
+P 3400 4000
+F 0 "F1" H 3400 4000 60  0000 C CNN
+F 1 "MF-MSMF050-2" H 3400 4100 60  0000 C CNN
+F 2 "Capacitors_SMD:C_1812_HandSoldering" H 3300 3900 60  0001 C CNN
+F 3 "https://www.bourns.com/PDFs/MFMSMF.pdf" H 3350 3700 60  0001 C CNN
+F 4 "0.00@0" H 3600 3800 60  0001 C CNN "Pricing"
+F 5 "1812 mils" H 3400 4400 60  0001 C CNN "Package ID"
+F 6 "Bournes" H 3400 4200 60  0001 C CNN "Manufacturer"
+F 7 "PTC Resettable Fuses" H 3400 4300 60  0001 C CNN "Description"
+	1    3400 4000
+	1    0    0    -1
+$EndComp
+Wire Wire Line
+	4650 2750 4400 2750
+Wire Wire Line
+	4400 2750 4400 2950
+Wire Wire Line
+	4400 2950 4150 2950
+Wire Wire Line
+	4650 2950 4650 2850
+Wire Wire Line
+	4650 2850 4300 2850
+Wire Wire Line
+	4300 2850 4300 2750
+Wire Wire Line
+	4300 2750 4150 2750
 $EndSCHEMATC

Commit message: before initial DRC
Connections:
- net GNDREF: now also U19.30 ((ADC13/OC1B/OC4B/PCINT13)PB6)
- net D+: now reaches P1.3 (D+), R30.2, Z1.1
- net D-: now reaches P1.2 (D-), R32.2, Z2.1
- net RESET: now reaches D2.2 (A), R33.2, SW1.2, U19.13 (~RESET~)
- net ENC-1: now reaches S1.1 (S1), U19.1 ((INT6/AIN0)PE6)
- net ENC-B: now reaches S1.5 (B), U19.20 ((RXD/INT2)PD2)
- net ENC-A: now reaches S1.3 (A), U19.27 ((T0/OC4D/ADC10)PD7)
- net USB-D-: now reaches R32.1, U19.3 (D-)
- net USB-D+: now reaches R30.1, U19.4 (D+)
- no-connect marks 20 -> 19
Changed lines of the file:
@@
 $EndComp
 $Comp
-L GNDREF #PWR0105
+L GNDREF #PWR0106
 U 1 1 580AC5C4
 P 3150 2750
-F 0 "#PWR0105" H 3150 2500 50  0001 C CNN
+F 0 "#PWR0106" H 3150 2500 50  0001 C CNN
 F 1 "GNDREF" H 3150 2600 50  0000 C CNN
 F 2 "" H 3150 2750 50  0000 C CNN
@@
 	3050 3900 3050 4250
 $Comp
-L GNDREF #PWR0106
+L GNDREF #PWR0107
 U 1 1 580AD10D
 P 4900 5600
-F 0 "#PWR0106" H 4900 5350 50  0001 C CNN
+F 0 "#PWR0107" H 4900 5350 50  0001 C CNN
 F 1 "GNDREF" H 4900 5450 50  0000 C CNN
 F 2 "" H 4900 5600 50  0000 C CNN
@@
 Connection ~ 5600 2050
 $Comp
-L GNDREF #PWR0107
+L GNDREF #PWR0108
 U 1 1 580AE22B
 P 6550 2050
-F 0 "#PWR0107" H 6550 1800 50  0001 C CNN
+F 0 "#PWR0108" H 6550 1800 50  0001 C CNN
 F 1 "GNDREF" H 6550 1900 50  0000 C CNN
 F 2 "" H 6550 2050 50  0000 C CNN
@@
 tx serial is used for \npotential serial LCD \ndisplay
 $Comp
-L GNDREF #PWR0108
+L GNDREF #PWR0109
 U 1 1 580B1F38
 P 8900 3800
-F 0 "#PWR0108" H 8900 3550 50  0001 C CNN
+F 0 "#PWR0109" H 8900 3550 50  0001 C CNN
 F 1 "GNDREF" H 8900 3650 50  0000 C CNN
 F 2 "" H 8900 3800 50  0000 C CNN
@@
 $EndComp
 $Comp
-L GNDREF #PWR0109
+L GNDREF #PWR0110
 U 1 1 580B1F98
 P 7800 3900
-F 0 "#PWR0109" H 7800 3650 50  0001 C CNN
+F 0 "#PWR0110" H 7800 3650 50  0001 C CNN
 F 1 "GNDREF" H 7800 3750 50  0000 C CNN
 F 2 "" H 7800 3900 50  0000 C CNN
@@
 	8900 3750 8900 3800
 $Comp
-L +5VP #PWR0110
+L +5VP #PWR0111
 U 1 1 580B2965
 P 5200 1100
-F 0 "#PWR0110" H 5200 950 50  0001 C CNN
+F 0 "#PWR0111" H 5200 950 50  0001 C CNN
 F 1 "+5VP" H 5200 1240 50  0000 C CNN
 F 2 "" H 5200 1100 50  0000 C CNN
@@
 NoConn ~ 6900 3250
 NoConn ~ 6900 3050
-NoConn ~ 6900 2950
 NoConn ~ 6900 2850
 NoConn ~ 6900 2750
@@
 Connection ~ 3050 3300
 $Comp
-L PWR_FLAG #FLG0111
+L PWR_FLAG #FLG0112
 U 1 1 580C0F96
 P 6200 2050
-F 0 "#FLG0111" H 6200 2145 50  0001 C CNN
+F 0 "#FLG0112" H 6200 2145 50  0001 C CNN
 F 1 "PWR_FLAG" H 6200 2230 50  0000 C CNN
 F 2 "" H 6200 2050 50  0000 C CNN
@@
 Connection ~ 6200 2050
 $Comp
-L PWR_FLAG #FLG0112
+L PWR_FLAG #FLG0113
 U 1 1 580C2BBD
 P 4650 2050
-F 0 "#FLG0112" H 4650 2145 50  0001 C CNN
+F 0 "#FLG0113" H 4650 2145 50  0001 C CNN
 F 1 "PWR_FLAG" H 4650 2230 50  0000 C CNN
 F 2 "" H 4650 2050 50  0000 C CNN
@@
 Wire Wire Line
 	4300 2750 4150 2750
+Text Label 4150 3700 0    60   ~ 0
+USB-D+
+Text Label 4250 3800 0    60   ~ 0
+USB-D-
+Text Label 3200 3800 0    60   ~ 0
+D-
+Text Label 3100 3700 0    60   ~ 0
+D+
+Text Label 7650 4550 0    60   ~ 0
+ENC-1
+Text Label 7650 4250 0    60   ~ 0
+ENC-A
+Text Label 7650 3750 0    60   ~ 0
+ENC-B
+Text Label 4500 2350 0    60   ~ 0
+RESET
+$Comp
+L GNDREF #PWR?
+U 1 1 5815DD38
+P 7000 2950
+F 0 "#PWR?" H 7000 2700 50  0001 C CNN
+F 1 "GNDREF" H 7000 2800 50  0000 C CNN
+F 2 "" H 7000 2950 50  0000 C CNN
+F 3 "" H 7000 2950 50  0000 C CNN
+	1    7000 2950
+	0    -1   -1   0
+$EndComp
+Wire Wire Line
+	6900 2950 7000 2950
 $EndSCHEMATC

Commit message: updating to new kicad version
Parts:
- P1: symbol USB_OTG -> USB_OTG-RESCUE-portable-line-mixer
Changed lines of the file:
@@
 EESchema Schematic File Version 2
+LIBS:portable-line-mixer-rescue
 LIBS:SW-Linear
 LIBS:SW-IQD
@@
 $EndComp
 $Comp
-L USB_OTG P1
+L USB_OTG-RESCUE-portable-line-mixer P1
 U 1 1 580C7DAA
 P 2750 3700
+AR Path="/580C7DAA" Ref="P1"  Part="1"
+AR Path="/580C77A2/580C7DAA" Ref="P1"  Part="1"
 F 0 "P1" H 3075 3575 50  0000 C CNN
 F 1 "USB_OTG" H 2750 3900 50  0000 C CNN
