File: audio-mixer.sch (KiCad schematic (older format))
At the start: 81 parts

Commit message: Updated Schematics
- added ethernet
- swapped to using prebuilt nano
- swapped to using db25 connector
- swapped other connectors
- added connectors for an LCD screen
Parts:
- removed C? (x2): 27pF, Capacitors_SMD:C_0805_HandSoldering, symbol Device:C_Small
- removed C? (x2): 47pF, Capacitors_SMD:C_0805_HandSoldering, symbol Device:C_Small
- removed C? (x2): 10uF, Capacitors_Tantalum_SMD:TantalC_SizeR_EIA-2012, symbol Device:CP_Small
- removed J?: JACK-TRS, SW-CUI-INC:SJ1-353XNG-3Pin, symbol SW-con:JACK-TRS
- removed U? (x4): RC4560, Housings_SSOP:TSSOP-8_4.4x3mm_Pitch0.65mm, symbol SW-texas-op_amps:RC4560
- added C25, C29: 1uF, SW-Kemet:Kemet_CAP_2220_5750Metric_D, symbol Device:C_Small
- added D1, D2, D3, D4, D5, D6, D7, D8: 0582BQ, SW-Semtech:SC-75_3L, symbol SW-Semtech:0582BQ
- added J3: Audio Out, SW-Hirose:DF11-4DP-2DSA, symbol Connector_Generic:Conn_02x02_Odd_Even
- added J4: Audio IN, SW-Hirose:DF11-24DP-2DSA, symbol Connector_Generic:Conn_02x12_Odd_Even
- added U3: OPA1604, Package_SSOP:TSSOP-14_4.4x5mm_P0.65mm, symbol SW-Texas:OPA1604
- C14, C15, C26, C27, C28, C32, C33, C34, C37, C38, C39, C42, C43, C44, C47, C48, C49, C52, C53, C54, C57, C58, C59, C62: renamed from C?; footprint Capacitors_SMD:C_0603_HandSoldering -> Capacitor_SMD:C_1206_3216Metric_Pad1.24x1.80mm_HandSolder
- R16, R17, R18, R19, R20, R21, R22, R23, R24, R25, R26, R27, R28, R29, R30, R31, R32, R33, R34, R35, R36, R37: renamed from R?; footprint Resistors_SMD:R_0805_HandSoldering -> Resistor_SMD:R_0603_1608Metric_Pad0.84x1.00mm_HandSolder
- U10, U11, U12, U13, U14, U4, U6, U7: renamed from U?; footprint Housings_SSOP:TSSOP-16_4.4x5mm_Pitch0.65mm -> Package_SSOP:TSSOP-16_4.4x5mm_P0.65mm
- gave numbers to parts that had none: 16
Connections:
- net labels added: -5VA
- net labels removed: +12VA, -12VA, -5V
- wire segments 402 -> 527
Other:
- note added: "Each input has jack, pot and summing resistor = 10k\n\n+-5VA = analog +5V, +5VD = digital +5V, (separate regulators)\nGNDREF = global ground"
- note removed: "Each input module has jack, pot and summing resistor = 10k\n\n+5VA = analog +5V, +5VD = digital +5V, (separate regulators)\n-5V, GNDREF = global ground"

Commit message: Added net labels and started schematic
Parts:
- added D9: 0582BQ, SW-Semtech:SC-75_3L, symbol SW-Semtech:0582BQ
- renumbered C14 to C21, C15 to C22, C16 to C23, U3 to U6, U4 to U7, U6 to U8, U7 to U9
Connections:
- net labels added: F-LIN-0, F-LIN-1, F-LIN-2, F-LIN-3, F-LIN-4, F-LIN-5, F-LIN-6, F-LIN-7, F-RIN-0, F-RIN-1, F-RIN-2, F-RIN-3, F-RIN-4, F-RIN-5, F-RIN-6, F-RIN-7, LINV, LOUT, LOUT-0, LOUT-1, LOUT-2, LOUT-3, LOUT-4, LOUT-5, LOUT-6, LOUT-7, RINV, ROUT, ROUT-0, ROUT-1, ROUT-2, ROUT-3, ROUT-4, ROUT-5, ROUT-6, ROUT-7
- wire segments 527 -> 533
