File: power_handling.sch (KiCad schematic (older format))
At the start: 89 parts, among them J1 Power In (Male-top), U1 LM27762, U2 74ACT32, U3 TS12A44514, U4 LMZ34002, U5 LM1085-12V, U6 TS12A44514, U7 74ACT32, U8 LM1085-5V, U9 LM27762

Commit message: Updated Schematics
- added ethernet
- swapped to using prebuilt nano
- swapped to using db25 connector
- swapped other connectors
- added connectors for an LCD screen
Parts:
- removed C14, C15, C16: 22uF, Capacitor_SMD:C_1206_3216Metric_Pad1.24x1.80mm_HandSolder, symbol Device:C_Small
- removed C? (x7): 10uF, Capacitors_Tantalum_SMD:TantalC_SizeR_EIA-2012, symbol Device:CP_Small
- removed C?: 22uF, Capacitors_Tantalum_SMD:TantalC_SizeB_EIA-3528_HandSoldering, symbol Device:CP_Small
- removed C? (x2): 1uF, Capacitors_SMD:C_0603_HandSoldering, symbol Device:C_Small
- removed C?: 0u1F, Capacitors_SMD:C_0603_HandSoldering, symbol Device:C_Small
- removed C?: 2u2F, Capacitors_SMD:C_1206_HandSoldering, symbol Device:C_Small
- removed C?: 1uF, Capacitors_SMD:C_0805_HandSoldering, symbol Device:C_Small
- removed C?: 2n2F, Capacitors_SMD:C_0805_HandSoldering, symbol Device:C_Small
- removed C?: 47pF, Capacitors_SMD:C_0805_HandSoldering, symbol Device:C_Small
- removed C?: 10uF, Capacitors_SMD:C_1206_HandSoldering, symbol Device:C_Small
- removed C? (x2): 0u01F, Capacitors_SMD:C_0603_HandSoldering, symbol Device:C_Small
- removed CON?: BARREL_JACK, SW-Switchcraft:L712RAS, symbol Connector_Generic:Conn_02x02_Odd_Even
- removed D?: CMMSH1-40, Diodes_SMD:SOD-123, symbol Device:D_Schottky_Small
- removed L?: 10uH, SW-Sumida:CDRH6D28, symbol Device:L_Small
- removed L?: 22uH, SW-Sumida:CDRH3D28NP, symbol Device:L_Small
- removed R?: 45k3, Resistors_SMD:R_0805_HandSoldering, symbol Device:R_Small
- removed R?: 147k, Resistors_SMD:R_0805_HandSoldering, symbol Device:R_Small
- removed R?: 10k, Resistors_SMD:R_0805_HandSoldering, symbol Device:R_Small
- removed R? (x2): 100R, Resistors_SMD:R_0603_HandSoldering, symbol Device:R_Small
- removed R?: 700R, Resistors_SMD:R_0603_HandSoldering, symbol Device:R_Small
- removed R?: 630R, Resistors_SMD:R_0603_HandSoldering, symbol Device:R_Small
- removed SW?: ON/OFF, SW-Eswitch:M7, symbol Switch:SW_SPST
- removed T? (x4): PMV45EN2, TO_SOT_Packages_SMD:SOT-23, symbol SW-NXP:PMV45EN2
- removed U1: LM27762, Package_SON:WSON-12-1EP_3x2mm_P0.5mm, symbol SW-Texas:LM27762
- removed U2, U7: 74ACT32, Package_SSOP:TSSOP-14_4.4x5mm_P0.65mm, symbol Logic_74xx:74LS32
- removed U3, U6: TS12A44514, Package_SSOP:TSSOP-14_4.4x5mm_P0.65mm, symbol SW-Texas:TS12A44514
- removed U4: LMZ34002, SW-Texas:RKG_(S-PB1QFN-N41), symbol SW-Texas:LMZ34002
- removed U? (x3): NCP1117ST50T3G_MountingTab, TO_SOT_Packages_SMD:SOT-223, symbol Regulator_Linear:NCP1117-5.0_SOT223
- removed U?: LT1085, TO_SOT_Packages_THT:TO-220_Neutral123_Horizontal_LargePads, symbol SW-Texas:LM1085
- removed U? (x2): MAX6820, TO_SOT_Packages_SMD:SOT-23-6_Handsoldering, symbol SW-dallas-semi-maxim:MAX6820
- removed U?: MAX1721, TO_SOT_Packages_SMD:SOT-23-6_Handsoldering, symbol SW-dallas-semi-maxim:MAX1721
- removed U?: LT3580, Housings_SSOP:MSOP-8-1EP_3x3mm_Pitch0.65mm, symbol SW-Linear:LT3580
- added T1: PMV45EN2, TO_SOT_Packages_SMD:SOT-23, symbol SW-NXP:PMV45EN2
- added U1: LM3880, Package_TO_SOT_SMD:SOT-23-6_Handsoldering, symbol SW-Texas:LM3880
- added U2: LTC3265, Package_SSOP:HTSSOP-20-1EP_4.4x6.5mm_P0.65mm_EP3.4x6.5mm_ThermalVias, symbol SW-Analog:LTC3265
- added U3: OPA1604, Package_SSOP:TSSOP-14_4.4x5mm_P0.65mm, symbol SW-Texas:OPA1604
- C1: value 2u2F -> 1uF; footprint Capacitor_SMD:C_0805_2012Metric_Pad1.15x1.50mm_HandSolder -> Capacitor_SMD:C_1206_3216Metric_Pad1.24x1.80mm_HandSolder; Manufacturer TDK -> (none); Manufacturer Part Number CGA4J3X7R1H225K125AE -> (none); Pricing 0.00@0 -> (none)
- C11, C8: value 0.1uF -> 10uF; footprint Capacitor_SMD:C_0805_2012Metric_Pad1.15x1.50mm_HandSolder -> Capacitor_SMD:C_1206_3216Metric_Pad1.24x1.80mm_HandSolder
- C12: value 0.1uF -> 0u1F; footprint Capacitor_SMD:C_0805_2012Metric_Pad1.15x1.50mm_HandSolder -> Capacitor_SMD:C_1206_3216Metric_Pad1.24x1.80mm_HandSolder
- C13: value 22uF -> 0u1F; Description Ceramic Capacitor -> (none); Manufacturer Murata -> (none); Manufacturer Part Number GRT31CR61E226KE01L -> (none); Pricing 0.00@0 -> (none)
- C19, C20, C21, C22, C23: footprint Capacitor_SMD:C_0805_2012Metric_Pad1.15x1.50mm_HandSolder -> Capacitor_SMD:C_1206_3216Metric_Pad1.24x1.80mm_HandSolder
- C2: value 0.47uF -> 1uF; footprint Capacitor_SMD:C_0805_2012Metric_Pad1.15x1.50mm_HandSolder -> Capacitor_SMD:C_1206_3216Metric_Pad1.24x1.80mm_HandSolder; Characteristics 10% -55ºC + 125ºC -> (none); Description Ceramic Capacitor -> (none); Manufacturer TDK -> (none); Manufacturer Part Number CGA4J3X7R1H474K125AE -> (none)
- C3: value 15uF -> 10uF; footprint Capacitor_SMD:C_0805_2012Metric_Pad1.15x1.50mm_HandSolder -> Capacitor_SMD:C_1206_3216Metric_Pad1.24x1.80mm_HandSolder; Characteristics X5R 1.669mΩ ESR -> (none); Description Ceramic Capacitor -> (none); Manufacturer TDK -> (none); Manufacturer Part Number C2012X5R1V156M125AC -> (none); Notes X5R 1.669mΩ ESR -> (none); Package ID 2012 metric -> (none); Pricing 0.00@0 -> (none)
- C4: value 2u2F -> 10uF; footprint Capacitor_SMD:C_0805_2012Metric_Pad1.15x1.50mm_HandSolder -> Capacitor_SMD:C_1206_3216Metric_Pad1.24x1.80mm_HandSolder; Manufacturer TDK -> (none); Manufacturer Part Number CGA4J3X7R1H225K125AE -> (none); Pricing 0.00@0 -> (none)
- C5: value 0.1uF -> 100nF; footprint Capacitor_SMD:C_0805_2012Metric_Pad1.15x1.50mm_HandSolder -> Capacitor_SMD:C_1206_3216Metric_Pad1.24x1.80mm_HandSolder
- C6: value 4u7F -> 100nF; footprint Capacitor_SMD:C_0805_2012Metric_Pad1.15x1.50mm_HandSolder -> Capacitor_SMD:C_1206_3216Metric_Pad1.24x1.80mm_HandSolder; Characteristics 10% -55ºC +85ºC -> (none); Manufacturer TDK -> (none); Manufacturer Part Number CGA4J3X5R1H475K125AB -> (none)
- C7: value 4u7F -> 10uF; footprint Capacitor_SMD:C_0805_2012Metric_Pad1.15x1.50mm_HandSolder -> Capacitor_SMD:C_1206_3216Metric_Pad1.24x1.80mm_HandSolder; Characteristics 10% -55ºC +85ºC -> (none); Manufacturer TDK -> (none); Manufacturer Part Number CGA4J3X5R1H475K125AB -> (none)
- R1: value 75kΩ -> 100kΩ; Characteristics 0.5% -55ºC +155ºC 1/8W -> (none); Description Thin Film Resistor -> (none); Manufacturer Vishay -> (none); Manufacturer Part Number MCT0603MD7502DP500 -> (none)
- R2, R3: value 68kΩ -> 100kΩ; Characteristics 0.1% -55ºC +155ºC 100mW -> (none); Description Thin Film Resistor -> (none); Manufacturer Vishay -> (none); Manufacturer Part Number TNPW060368K0BEEA -> (none)
- R4: value 174kΩ -> 681kΩ; Characteristics 0.1% -55ºC +155ºC 100mW -> (none); Description Thin Film Resistor -> (none); Manufacturer Vishay -> (none); Manufacturer Part Number TNPW0603174KBEEA -> (none); Package ID 1608 metric -> (none); Pricing 0.00@0 -> (none)
- R5: Characteristics 0.5% -55ºC +155ºC 1/8W -> (none); Description Thin Film Resistor -> (none); Manufacturer Vishay -> (none); Manufacturer Part Number MCT0603MD7502DP500 -> (none)
- R6: value 22.6kΩ -> 75kΩ; Characteristics 0.1% -55ºC +155ºC 100mW -> (none); Description Thin Film Resistor -> (none); Manufacturer Vishay -> (none); Manufacturer Part Number TNPW060322K6BEEA -> (none); Package ID 1608 metric -> (none); Pricing 0.00@0 -> (none)
- R8: value 143kΩ -> 681kΩ; Characteristics 0.1% -55ºC +155ºC 100mW -> (none); Description Thin Film Resistor -> (none); Manufacturer Vishay -> (none); Manufacturer Part Number TNPW0603143KBEEA -> (none); Package ID 1608 metric -> (none); Pricing 0.00@0 -> (none)
Connections:
- net labels added: Audio_Power_Enable
- net labels removed: +2V5, +5VP, -2.5V, -5V
- wire segments 389 -> 184
- no-connect marks 3 -> 0
Other:
- note added: "+12V is main supply\n+5V is unswitched digital supply\n+-5VA is switched analog supply for pots\n+5VD is switched digital supply for pots\n+- 12VA is switched analog supply for op amp"
- note added: "Power Supply Sequencing\n\n+12V on first\n+5V on next (no control)\n+-5VA on next (first flag)\n+5VD on next (second flag)\n+-12VA on next (third flag)"
- note added: "RT=GND=> 500kHz switching frequency"
- note added: "V+-=1.2V* (R1/R2 +1)\n12.09 ~~= 1.2V* (681k/75k + 1)"
- note removed: "+12V -> -12V conversion"
- note removed: "+12V is regulated +12V@5A DC supply. \n+5V is 5V@3A supply\n\n\n+12VA is positive supply for op amps used as audio amplifiers\n-12VA is negative supply for op amps used as audio amplifiers\n+5VA is positive analog supply for potentiometer chips\n-5VA is negative analog supply for potentiometer chips\n+2.5V is positive supply for audio switch chips and io \nexpanders at that logic level\n-2.5V is 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"
- note removed: "+5V -> -5V conversion"
- note removed: "0-5V control signal switch/mux chips will use 5V as power\n\naudio signal switch chips will use \n+2.5VA as positive rail\n-2.5VA as negative rail\n\nPotentiometers use \n5V as digital power\n5VA as analog positive rail\n-5VA as negative analog rail\n\nop amps use \n+12VA as analog positive rail\n-12VA as analog negative rail\n\nfor each chip voltage level, i2c lines are pulled to \nthe individua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"
- note removed: "12V DC output regulator"
- note removed: "2u2F cap = 25V X5R, 1206\n10uF cap = 25V X5R, 1206\n1uF cap = 50V X5R, 0805\nDiode = Central Semi CMMSH1-40\n10uH = SUMIDA CDRH6D28NP-100NC\n22uH = SUMIDA CDRH6D28NP-220NC"
- note removed: "88uF total capacitance"
- note removed: "Main Power Supplies"
- note removed: "Power connections for MUX"
- note removed: "Power for 7400 series OR gates"
- note removed: "Power sequence:\n1) +5VA, -5V\n2) +5VP, +5VD\n3) +12VA, -12VA"
- note removed: "Provides -12V supply for op amps"
- note removed: "Provides ±2.5 supply for\naudio muxes, switches\nand related IO expanders\nIout = 250mA max \nAssume Iin = 500mA max"
- note removed: "Rtop = Rbottom ((VTRIP / 0.618) - 1) \n"
- note removed: "Vout = 1.2V * (R1+R2)/R2\n2.52 ~~= 1.2V * (75k + 68k)/68k \nusing E24 values\n\ncaps need low ESR\nuse X7R or X5R\nceramic SMD caps\n"
- note removed: "tDELAY (s) = 2.48 s/Farad * (10^6) * CSET (F)\nuF as CSET will get seconds\n!Verify before production!"
- moved on the sheet: C10, C17, C18, C19, C20, C21, C22, C23, C9

Commit message: Added net labels and started schematic
Parts:
- renumbered C19 to C1, C1 to C10, C2 to C11, C3 to C12, C4 to C13, C5 to C14, C6 to C15, C7 to C16, C8 to C17, C11 to C18, C12 to C19, C20 to C2, C13 to C20, C21 to C3, C22 to C4, C23 to C5, C9 to C6, C10 to C7, C17 to C8, C18 to C9, R10 to R1, R4 to R10, R5 to R11, R6 to R12, R8 to R13, R11 to R2, R1 to R3, R2 to R4, R3 to R5, R12 to R6, R13 to R7, R7 to R8, U9 to U1, U1 to U2, U5 to U3, U8 to U4, U2 to U5, U3 to U6
Connections:
- net labels added: +5VD_EN, ±12VA_EN, ±5VA_EN

Commit message: Swapped encoder for connector
Parts:
- T1: footprint TO_SOT_Packages_SMD:SOT-23 -> Package_TO_SOT_SMD:SOT-23
Changed lines of the file:
@@
 F 0 "T1" H 5541 2254 50  0000 L CNN
 F 1 "PMV45EN2" H 5541 2345 50  0000 L CNN
-F 2 "TO_SOT_Packages_SMD:SOT-23" H 5550 2850 50  0001 C CNN
+F 2 "Package_TO_SOT_SMD:SOT-23" H 5550 2850 50  0001 C CNN
 F 3 "http://cache.nxp.com/documents/data_sheet/PMV45EN2.pdf?pspll=1" H 5800 2000 50  0001 C CNN
-F 4 "0.00@0" H 5150 2550 60  0001 C CNN "Pricing"
-F 5 "30V 5.1A" H 5600 2950 60  0001 C CNN "Characteristics"
+F 4 "30V 5.1A" H 5600 2950 60  0001 C CNN "Characteristics"
+F 5 "NXP" H 5850 2550 60  0001 C CNN "Manufacturer"
 F 6 "N-channel Trench MOSFET" H 5950 2650 60  0001 C CNN "Description"
-F 7 "NXP" H 5850 2550 60  0001 C CNN "Manufacturer"
-F 8 "SOT23" H 6050 2750 60  0001 C CNN "Package ID"
+F 7 "SOT23" H 6050 2750 60  0001 C CNN "Package ID"
+F 8 "0.00@0" H 5150 2550 60  0001 C CNN "Pricing"
 	1    5350 2300
 	1    0    0    1

Commit message: Portable Line Mixer done
Parts:
- U1: footprint Package_SON:WSON-12-1EP_3x2mm_P0.5mm -> SW-Package-SON:WSON-12-1EP_3x2mm_P0.5mm
- U5: footprint Package_SSOP:HTSSOP-20-1EP_4.4x6.5mm_P0.65mm_EP3.4x6.5mm_ThermalVias -> SW-Linear:TSSOP-20-1EP_4.4x6.5mm_P0.65mm_EP2.75x6.07mm-LTC3265; Pricing (none) -> 0.00@0
Connections:
- net labels added: ADJ+, ADJ-, BYP+, BYP-, CBST+, CBST-, CINV+, CINV-, VOUT+, VOUT-
Changed lines of the file:
@@
 F 0 "U1" H 8450 2647 60  0000 C CNN
 F 1 "LM27762" H 8450 2541 60  0000 C CNN
-F 2 "Package_SON:WSON-12-1EP_3x2mm_P0.5mm" H 8250 2650 60  0001 C CNN
+F 2 "SW-Package-SON:WSON-12-1EP_3x2mm_P0.5mm" H 8250 2650 60  0001 C CNN
 F 3 "http://www.ti.com/lit/ds/symlink/lm27762.pdf" H 8450 2850 60  0001 C CNN
 F 4 "Vin 2.7V to 5.5V, Vout ±1.5 to 5V, ±250mA Iout, 2MHz switching frequency," H 8550 2950 60  0001 C CNN "Characteristics"
@@
 F 0 "U5" H 8325 3628 50  0000 C CNN
 F 1 "LTC3265" H 8325 3537 50  0000 C CNN
-F 2 "Package_SSOP:HTSSOP-20-1EP_4.4x6.5mm_P0.65mm_EP3.4x6.5mm_ThermalVias" H 8300 4700 50  0001 C CNN
+F 2 "SW-Linear:TSSOP-20-1EP_4.4x6.5mm_P0.65mm_EP2.75x6.07mm-LTC3265" H 8300 4700 50  0001 C CNN
 F 3 "http://www.analog.com/media/en/technical-documentation/data-sheets/3265fa.pdf" H 8300 4700 50  0001 C CNN
+F 4 "0.00@0" H 8300 4700 50  0001 C CNN "Pricing"
 	1    8300 4700
 	1    0    0    -1
@@
 Text Label 4850 2300 0    50   ~ 0
 +5VD_EN
+Text Label 8050 3900 1    50   ~ 0
+CBST+
+Text Label 8250 3900 1    50   ~ 0
+CBST-
+Text Label 8400 3900 1    50   ~ 0
+CINV+
+Text Label 8600 3900 1    50   ~ 0
+CINV-
+Text Label 8900 4700 0    50   ~ 0
+ADJ+
+Text Label 8900 5100 0    50   ~ 0
+ADJ-
+Text Label 7700 5450 0    50   ~ 0
+BYP+
+Text Label 7750 5050 2    50   ~ 0
+BYP-
+Text Label 8900 5650 0    50   ~ 0
+VOUT-
+Text Label 7700 5600 3    50   ~ 0
+VOUT+
 $EndSCHEMATC
