File: ard-nano-hdr-ethernet.sch (KiCad schematic (older format))
At the start: 7 parts, among them SW1 Nano Reset, SW2 I2C Reset, SW3 SPST Reset

Commit message: Updated Schematics
- added ethernet
- swapped to using prebuilt nano
- swapped to using db25 connector
- swapped other connectors
- added connectors for an LCD screen
Parts:
- removed SW2: I2C Reset, SW-Eswitch:TL1105WF, symbol SW-gElectroMech:SPST_MOM_SHLD
- removed SW3: SPST Reset, SW-Eswitch:TL1105WF, symbol SW-gElectroMech:SPST_MOM_SHLD
- added J2: LCD Connection I2C, SW-Hirose:DF11-4DP-2DSA, symbol Connector_Generic:Conn_02x02_Odd_Even
- R14, R15: renamed from R?; footprint Capacitors_SMD:C_0805_HandSoldering -> Resistor_SMD:R_0603_1608Metric_Pad0.84x1.00mm_HandSolder
- gave numbers to parts that had none: 1
Connections:
- net labels added: Audio_Power_EN
- net labels removed: +5VD, D2_SPST, D3_I2C, D5_INT, I2C_RST, IO_EXP_INT, SCL, SDA, SPST_RST
- wire segments 55 -> 53
- no-connect marks 19 -> 18
Other:
- note added: "D0 -\nD1 -\nD2 - External Interrupt - ENC-B - Pullup\nD3 - External Interrupt - ENC-SW -Pullup\nD4 - MicroSD slave select\nD5 - ENC-A - pullup\nD6 - Audio Power Enable\nD7\nD8\nD9\nD10 - Ethernet Slave Select\nD11 - MOSI\nD12 - MISO\n\nUse D2 and D3 as interupts for encoder,\n1 for detecting switch and one for\ndetecting transition which is less \nimportant so only 1/2 accuacy is acceptable.\nOth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"
- note added: "Make sure to remove pullup resistors off of LCD board (R6, R7 I think)"
- note removed: "Use D0(PD2) and D7(PE6) as interupts for encoder,\n1 for detecting switch and one for\ndetecting transition which is less \nimportant so only 1/2 accuacy is acceptable.\nOther encoder pin is connected to D6(PD7)\nMake certain to turn on pullup resistors on\nthese pins as they will be pulled low on\nchange."
- note removed: "tx serial is used for \npotential serial LCD \ndisplay"

Commit message: Swapped encoder for connector
Parts:
- removed S1: PEC11-4215F-S24, SW-Bournes:PEC11R-4xxx-Sxxxx, symbol SW-Bournes-Pro-Audio:PEC11-4215F-S24
- added J5: Encoder Connection, SW-Hirose:DF11-4DP-2DSA, symbol Connector_Generic:Conn_02x02_Odd_Even
Other:
- note added: "Use PEC11-4215F-S24\nEncoder.\nSolder + Heatshrink wires\nUse APM Hexseal sealed nut"
Changed lines of the file:
@@
 	6400 2300 6400 2450
 Connection ~ 6400 2450
-$Comp
-L SW-Bournes-Pro-Audio:PEC11-4215F-S24 S1
-U 1 1 5AC62149
-P 1750 2500
-F 0 "S1" H 1750 2650 60  0000 C CNN
-F 1 "PEC11-4215F-S24" H 1750 2300 60  0000 C CNN
-F 2 "SW-Bournes:PEC11R-4xxx-Sxxxx" H 1650 2550 60  0001 C CNN
-F 3 "http://www.bourns.com/docs/Product-Datasheets/pec11R.pdf" H 1600 2850 60  0001 C CNN
-F 4 "0.00@0" H 2050 3150 60  0001 C CNN "Pricing"
-F 5 "Bournes Pro Audio" H 1750 2950 60  0001 C CNN "Manufacturer"
-F 6 "PEC11R Series - 12 mm Incremental Encoder" H 1750 3050 60  0001 C CNN "Description"
-	1    1750 2500
-	1    0    0    1
-$EndComp
 Text Notes 1700 5650 0    60   ~ 0
 D0 -\nD1 -\nD2 - External Interrupt - ENC-B - Pullup\nD3 - External Interrupt - ENC-SW -Pullup\nD4 - MicroSD slave select\nD5 - ENC-A - pullup\nD6 - Audio Power Enable\nD7\nD8\nD9\nD10 - Ethernet Slave Select\nD11 - MOSI\nD12 - MISO\n\nUse D2 and D3 as interupts for encoder,\n1 for detecting switch and one for\ndetecting transition which is less \nimportant so only 1/2 accuacy is acceptable.\nOther encoder pin is connected to D5\nMake certain to turn on pullup resistors on\nthese pins as they will be pulled low on\nchange.
-Wire Wire Line
-	3100 2450 2050 2450
 Wire Wire Line
 	1400 2550 1400 3250
@@
 	-1   0    0    -1
 $EndComp
-$Comp
-L power:GNDREF #PWR029
-U 1 1 5AC62165
-P 2200 2600
-F 0 "#PWR029" H 2200 2350 50  0001 C CNN
-F 1 "GNDREF" H 2200 2450 50  0000 C CNN
-F 2 "" H 2200 2600 50  0000 C CNN
-F 3 "" H 2200 2600 50  0000 C CNN
-	1    2200 2600
-	-1   0    0    -1
-$EndComp
-Wire Wire Line
-	2050 2500 2200 2500
-Wire Wire Line
-	2200 2500 2200 2600
-Wire Wire Line
-	1400 2450 1100 2450
 Wire Wire Line
 	1100 2450 1100 2500
@@
 	7200 4050 6400 4050
 Connection ~ 6400 4050
+$Comp
+L Connector_Generic:Conn_02x02_Odd_Even J5
+U 1 1 5AFC62E7
+P 1650 2450
+F 0 "J5" H 1700 2550 50  0000 C CNN
+F 1 "Encoder Connection" H 1700 2250 50  0000 C CNN
+F 2 "SW-Hirose:DF11-4DP-2DSA" H 1650 2450 50  0001 C CNN
+F 3 "~" H 1650 2450 50  0001 C CNN
+	1    1650 2450
+	1    0    0    -1
+$EndComp
+Wire Wire Line
+	1100 2450 1450 2450
+Wire Wire Line
+	1400 2550 1450 2550
+Wire Wire Line
+	1950 2450 3100 2450
+Wire Wire Line
+	1950 2550 2050 2550
+Text Notes 1450 2150 0    50   ~ 0
+Use PEC11-4215F-S24\nEncoder.\nSolder + Heatshrink wires\nUse APM Hexseal sealed nut
 $EndSCHEMATC

Commit message: Portable Line Mixer done
Connections:
- wire segments 53 -> 57
Changed lines of the file:
@@
 Text Notes 3950 1850 0    60   ~ 0
 Pins D4, D10, D11, D12, D13 are \nused by gravitech.us ethernet card\nEthernet and USB connections are \nprovided by short cables to \nexternal connectors
-Text HLabel 6900 2950 2    60   BiDi ~ 0
+Text HLabel 7450 2950 2    60   BiDi ~ 0
 5V-SDA
-Text HLabel 6900 2850 2    60   Output ~ 0
+Text HLabel 7450 2850 2    60   Output ~ 0
 5V-SCL
 Text Label 5750 2450 0    60   ~ 0
@@
 	5650 4050 6400 4050
 Wire Wire Line
-	6400 2450 6400 4050
+	6400 2450 6400 3250
 $Comp
 L SW-gElectroMech:SPST_MOM_SHLD SW1
@@
 Text Notes 1700 5650 0    60   ~ 0
 D0 -\nD1 -\nD2 - External Interrupt - ENC-B - Pullup\nD3 - External Interrupt - ENC-SW -Pullup\nD4 - MicroSD slave select\nD5 - ENC-A - pullup\nD6 - Audio Power Enable\nD7\nD8\nD9\nD10 - Ethernet Slave Select\nD11 - MOSI\nD12 - MISO\n\nUse D2 and D3 as interupts for encoder,\n1 for detecting switch and one for\ndetecting transition which is less \nimportant so only 1/2 accuacy is acceptable.\nOther encoder pin is connected to D5\nMake certain to turn on pullup resistors on\nthese pins as they will be pulled low on\nchange.
-Wire Wire Line
-	1400 2550 1400 3250
-Wire Wire Line
-	1400 3250 3100 3250
 Wire Wire Line
 	2050 2950 2050 2550
@@
 Wire Wire Line
 	1100 2450 1100 2500
-Text Label 2350 3250 2    60   ~ 0
+Text Label 2750 2750 2    60   ~ 0
 ENC-1
 Text Label 2350 2950 2    60   ~ 0
 ENC-A
-Text Label 2350 2450 2    60   ~ 0
+Text Label 3000 2450 2    60   ~ 0
 ENC-B
 $Comp
@@
 	2050 2950 4150 2950
 Wire Wire Line
-	3100 3250 3100 2750
-Wire Wire Line
-	3100 2750 4150 2750
-Wire Wire Line
 	3700 3050 4150 3050
 Wire Wire Line
@@
 Connection ~ 5900 2850
 Wire Wire Line
-	5900 2850 6650 2850
-Wire Wire Line
 	5750 2600 5750 2550
 Connection ~ 5750 2550
@@
 L Connector_Generic:Conn_02x02_Odd_Even J2
 U 1 1 5E3F25AA
-P 6900 3150
-F 0 "J2" H 6950 3250 50  0000 C CNN
-F 1 "LCD Connection I2C" H 6950 2950 50  0000 C CNN
-F 2 "SW-Hirose:DF11-4DP-2DSA" H 6900 3150 50  0001 C CNN
-F 3 "~" H 6900 3150 50  0001 C CNN
-	1    6900 3150
-	1    0    0    -1
-$EndComp
-Wire Wire Line
-	6550 2950 6550 3250
-Wire Wire Line
-	6550 3250 6700 3250
+P 7000 3250
+F 0 "J2" H 7050 3350 50  0000 C CNN
+F 1 "LCD Connection I2C" H 7050 3050 50  0000 C CNN
+F 2 "SW-Hirose:DF11-4DP-2DSA" H 7000 3250 50  0001 C CNN
+F 3 "~" H 7000 3250 50  0001 C CNN
+	1    7000 3250
+	-1   0    0    1
+$EndComp
+Wire Wire Line
+	6550 2950 6550 3150
+Wire Wire Line
+	6550 3150 6700 3150
 Connection ~ 6550 2950
 Wire Wire Line
-	6550 2950 6900 2950
-Wire Wire Line
-	6650 2850 6650 3150
-Wire Wire Line
-	6650 3150 6700 3150
-Connection ~ 6650 2850
-Wire Wire Line
-	6650 2850 6900 2850
+	6550 2950 7450 2950
 $Comp
 L power:+5V #PWR030
 U 1 1 5E3F4B75
-P 7450 3150
-F 0 "#PWR030" H 7450 3000 50  0001 C CNN
-F 1 "+5V" H 7465 3323 50  0000 C CNN
-F 2 "" H 7450 3150 50  0001 C CNN
-F 3 "" H 7450 3150 50  0001 C CNN
-	1    7450 3150
-	1    0    0    -1
-$EndComp
-Wire Wire Line
-	7200 3150 7450 3150
-Wire Wire Line
-	7200 3250 7200 4050
-Wire Wire Line
-	7200 4050 6400 4050
-Connection ~ 6400 4050
+P 7750 3250
+F 0 "#PWR030" H 7750 3100 50  0001 C CNN
+F 1 "+5V" H 7765 3423 50  0000 C CNN
+F 2 "" H 7750 3250 50  0001 C CNN
+F 3 "" H 7750 3250 50  0001 C CNN
+	1    7750 3250
+	1    0    0    -1
+$EndComp
+Wire Wire Line
+	7200 3250 7750 3250
 $Comp
 L Connector_Generic:Conn_02x02_Odd_Even J5
 U 1 1 5AFC62E7
-P 1650 2450
-F 0 "J5" H 1700 2550 50  0000 C CNN
-F 1 "Encoder Connection" H 1700 2250 50  0000 C CNN
-F 2 "SW-Hirose:DF11-4DP-2DSA" H 1650 2450 50  0001 C CNN
-F 3 "~" H 1650 2450 50  0001 C CNN
-	1    1650 2450
-	1    0    0    -1
-$EndComp
-Wire Wire Line
-	1100 2450 1450 2450
+P 1750 2450
+F 0 "J5" H 1800 2550 50  0000 C CNN
+F 1 "Encoder Connection" H 1800 2250 50  0000 C CNN
+F 2 "SW-Hirose:DF11-4DP-2DSA" H 1750 2450 50  0001 C CNN
+F 3 "~" H 1750 2450 50  0001 C CNN
+	1    1750 2450
+	-1   0    0    -1
+$EndComp
 Wire Wire Line
 	1400 2550 1450 2550
-Wire Wire Line
-	1950 2450 3100 2450
 Wire Wire Line
 	1950 2550 2050 2550
 Text Notes 1450 2150 0    50   ~ 0
 Use PEC11-4215F-S24\nEncoder.\nSolder + Heatshrink wires\nUse APM Hexseal sealed nut
+Wire Wire Line
+	3100 2450 2450 2450
+Wire Wire Line
+	2450 2450 2450 2250
+Wire Wire Line
+	2450 2250 800  2250
+Wire Wire Line
+	800  2250 800  2750
+Wire Wire Line
+	2250 2750 2250 2450
+Wire Wire Line
+	2250 2450 1950 2450
+Wire Wire Line
+	2250 2750 4150 2750
+Wire Wire Line
+	1400 2750 1400 2550
+Wire Wire Line
+	800  2750 1400 2750
+Wire Wire Line
+	7350 2850 7350 3150
+Wire Wire Line
+	7350 3150 7200 3150
+Connection ~ 7350 2850
+Wire Wire Line
+	7350 2850 7450 2850
+Wire Wire Line
+	5900 2850 7350 2850
+Wire Wire Line
+	6400 3250 6700 3250
+Connection ~ 6400 3250
+Wire Wire Line
+	6400 3250 6400 4050
+Wire Wire Line
+	1100 2450 1450 2450
 $EndSCHEMATC

Commit message: Swapped right angle reset switch for straight
Parts:
- removed SW1: Nano Reset, SW-Eswitch:TL1105WF, symbol SW-gElectroMech:SPST_MOM_SHLD
- added SW1: Nano Reset, SW-Eswitch:TL1105, symbol SW-gElectroMech:SPST_MOM
Connections:
- wire segments 57 -> 54
Changed lines of the file:
@@
 Wire Wire Line
 	6400 2450 6400 3250
-$Comp
-L SW-gElectroMech:SPST_MOM_SHLD SW1
-U 1 1 5AB58C6D
-P 6200 2450
-F 0 "SW1" H 6200 2750 50  0000 C CNN
-F 1 "Nano Reset" H 6200 2650 50  0000 C CNN
-F 2 "SW-Eswitch:TL1105WF" H 6200 2650 50  0001 C CNN
-F 3 "" H 6200 2650 50  0001 C CNN
-	1    6200 2450
-	1    0    0    -1
-$EndComp
-Wire Wire Line
-	6000 2400 6000 2300
-Wire Wire Line
-	6000 2300 6400 2300
-Wire Wire Line
-	6400 2300 6400 2450
-Connection ~ 6400 2450
 Text Notes 1700 5650 0    60   ~ 0
 D0 -\nD1 -\nD2 - External Interrupt - ENC-B - Pullup\nD3 - External Interrupt - ENC-SW -Pullup\nD4 - MicroSD slave select\nD5 - ENC-A - pullup\nD6 - Audio Power Enable\nD7\nD8\nD9\nD10 - Ethernet Slave Select\nD11 - MOSI\nD12 - MISO\n\nUse D2 and D3 as interupts for encoder,\n1 for detecting switch and one for\ndetecting transition which is less \nimportant so only 1/2 accuacy is acceptable.\nOther encoder pin is connected to D5\nMake certain to turn on pullup resistors on\nthese pins as they will be pulled low on\nchange.
@@
 Wire Wire Line
 	1100 2450 1450 2450
+$Comp
+L SW-gElectroMech:SPST_MOM SW1
+U 1 1 5AC3DFC3
+P 6200 2450
+F 0 "SW1" H 6200 2750 50  0000 C CNN
+F 1 "Nano Reset" H 6200 2650 50  0000 C CNN
+F 2 "SW-Eswitch:TL1105" H 6200 2650 50  0001 C CNN
+F 3 "" H 6200 2650 50  0001 C CNN
+F 4 "0.00@0" H 6200 2450 50  0001 C CNN "Pricing"
+	1    6200 2450
+	1    0    0    -1
+$EndComp
 $EndSCHEMATC
